File: flipper black PCB/Flipper black ki cad/.history/Flipper black ki cad.kicad_sch (KiCad schematic)
At the start: 226 parts, among them J1 Barrel_Jack, J2 Value: DISP_3.5_WAVESHARE, P1 JST-2pin, P2 USB_C_Plug_USB2.0, Q1 MMBT2222A, Q2 FS8205A, SW1 SW_Push, SW2 SW_Push, U1 ESP32-S3, U10 BGA725L6, U11 TLV70018_SOT23-5, U12 TXB0102DCU, U13 MCP23017x-x-SS, U14 TSOP382xx, U15 TP4056, U17 AP2112K-3.3, U18 DW01A, U2 W25Q128JVS, U3 CC1101, U4 SX1276, U5 PE4259, U6 PE4259, U7 PN5321A3HN, U8 MAX-M8Q, U9 MASW-007221, X1 B3715 868MHz SAW Filter, X2 B3715 868MHz SAW Filter, Y1 40MHz SMD 3225, Y2 26 MHz SMD, Y3 32 MHz SMD, Y4 27.120 MHz

Commit message: lol
Parts:
- removed R37, R38: 100R, symbol Device:R
- added SW3, SW4, SW5, SW6, SW7, SW8: SW_Push, symbol Switch:SW_Push
Connections:
- net +5V: now also U18.2 (CS)
- net at C101.1, P1.1, U18.5 (VCC): now also U15.5 (BAT)
Other:
- note added: "AP2112K"
- note added: "BUTTON"
- moved on the sheet: C72, C87, IR_LEDs1, IR_LEDs2, IR_LEDs3, P2, Q1, R29, R30, R31, R32, R40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

Commit message: suii
Parts:
- SW3: value SW_Push -> BTN_POWER
- SW4: value SW_Push -> BTN_OK
- SW5: value SW_Push -> BTN_UP
- SW6: value SW_Push -> BTN_DOWN
- SW7: value SW_Push -> BTN_LEFT
- SW8: value SW_Push -> BTN_RIGHT
Other:
- moved on the sheet: SW3, SW4, SW5, SW6, SW7, SW8
Changed lines of the file:
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@@
 	(polyline
 		(pts
-			(xy 515.62 434.34) (xy 617.22 434.34)
+			(xy 515.62 434.34) (xy 632.46 434.34)
 		)
 		(stroke
@@
 	(polyline
 		(pts
-			(xy 515.62 345.44) (xy 617.22 345.44)
+			(xy 515.62 345.44) (xy 632.46 345.44)
 		)
 		(stroke
@@
 	(wire
 		(pts
+			(xy 546.1 373.38) (xy 546.1 384.81)
+		)
+		(stroke
+			(width 0)
+			(type default)
+		)
+	)
+	(wire
+		(pts
 			(xy 196.85 173.99) (xy 209.55 173.99)
 		)
@@
 	(wire
 		(pts
+			(xy 539.75 373.38) (xy 546.1 373.38)
+		)
+		(stroke
+			(width 0)
+			(type default)
+		)
+	)
+	(wire
+		(pts
 			(xy 163.83 273.05) (xy 163.83 279.4)
 		)
@@
 	(polyline
 		(pts
-			(xy 617.22 434.34) (xy 617.22 345.44)
+			(xy 632.46 434.34) (xy 632.46 345.44)
 		)
 		(stroke
@@
 	(symbol
 		(lib_id "Switch:SW_Push")
-		(at 566.42 401.32 0)
+		(at 570.23 401.32 0)
 		(unit 1)
 		(body_style 1)
@@
 		(fields_autoplaced yes)
 		(property "Reference" "SW7"
-			(at 566.42 393.7 0)
+			(at 570.23 393.7 0)
 			(show_name no)
 			(do_not_autoplace no)
@@
 			)
 		)
-		(property "Value" "SW_Push"
-			(at 566.42 396.24 0)
+		(property "Value" "BTN_LEFT"
+			(at 570.23 396.24 0)
 			(show_name no)
 			(do_not_autoplace no)
@@
 		)
 		(property "Footprint" ""
-			(at 566.42 396.24 0)
+			(at 570.23 396.24 0)
 			(hide yes)
 			(show_name no)
@@
 		)
 		(property "Datasheet" ""
-			(at 566.42 396.24 0)
+			(at 570.23 396.24 0)
 			(hide yes)
 			(show_name no)
@@
 		)
 		(property "Description" "Push button switch, generic, two pins"
-			(at 566.42 401.32 0)
+			(at 570.23 401.32 0)
 			(hide yes)
 			(show_name no)
@@
 	(symbol
 		(lib_id "Switch:SW_Push")
-		(at 595.63 401.32 0)
+		(at 603.25 401.32 0)
 		(unit 1)
 		(body_style 1)
@@
 		(fields_autoplaced yes)
 		(property "Reference" "SW8"
-			(at 595.63 393.7 0)
+			(at 603.25 393.7 0)
 			(show_name no)
 			(do_not_autoplace no)
@@
 			)
 		)
-		(property "Value" "SW_Push"
-			(at 595.63 396.24 0)
+		(property "Value" "BTN_RIGHT"
+			(at 603.25 396.24 0)
 			(show_name no)
 			(do_not_autoplace no)
@@
 		)
 		(property "Footprint" ""
-			(at 595.63 396.24 0)
+			(at 603.25 396.24 0)
 			(hide yes)
 			(show_name no)
@@
 		)
 		(property "Datasheet" ""
-			(at 595.63 396.24 0)
+			(at 603.25 396.24 0)
 			(hide yes)
 			(show_name no)
@@
 		)
 		(property "Description" "Push button switch, generic, two pins"
-			(at 595.63 401.32 0)
+			(at 603.25 401.32 0)
 			(hide yes)
 			(show_name no)
@@
 	(symbol
 		(lib_id "Switch:SW_Push")
-		(at 539.75 373.38 0)
+		(at 534.67 373.38 0)
 		(unit 1)
 		(body_style 1)
@@
 		(fields_autoplaced yes)
 		(property "Reference" "SW3"
-			(at 539.75 365.76 0)
+			(at 534.67 365.76 0)
 			(show_name no)
 			(do_not_autoplace no)
@@
 			)
 		)
-		(property "Value" "SW_Push"
-			(at 539.75 368.3 0)
+		(property "Value" "BTN_POWER"
+			(at 534.67 368.3 0)
 			(show_name no)
 			(do_not_autoplace no)
@@
 		)
 		(property "Footprint" ""
-			(at 539.75 368.3 0)
+			(at 534.67 368.3 0)
 			(hide yes)
 			(show_name no)
@@
 		)
 		(property "Datasheet" ""
-			(at 539.75 368.3 0)
+			(at 534.67 368.3 0)
 			(hide yes)
 			(show_name no)
@@
 		)
 		(property "Description" "Push button switch, generic, two pins"
-			(at 539.75 373.38 0)
+			(at 534.67 373.38 0)
 			(hide yes)
 			(show_name no)
@@
 	(symbol
 		(lib_id "Switch:SW_Push")
-		(at 539.75 401.32 0)
+		(at 534.67 401.32 0)
 		(unit 1)
 		(body_style 1)
@@
 		(fields_autoplaced yes)
 		(property "Reference" "SW6"
-			(at 539.75 393.7 0)
+			(at 534.67 393.7 0)
 			(show_name no)
 			(do_not_autoplace no)
@@
 			)
 		)
-		(property "Value" "SW_Push"
-			(at 539.75 396.24 0)
+		(property "Value" "BTN_DOWN"
+			(at 534.67 396.24 0)
 			(show_name no)
 			(do_not_autoplace no)
@@
 		)
 		(property "Footprint" ""
-			(at 539.75 396.24 0)
+			(at 534.67 396.24 0)
 			(hide yes)
 			(show_name no)
@@
 		)
 		(property "Datasheet" ""
-			(at 539.75 396.24 0)
+			(at 534.67 396.24 0)
 			(hide yes)
 			(show_name no)
@@
 		)
 		(property "Description" "Push button switch, generic, two pins"
-			(at 539.75 401.32 0)
+			(at 534.67 401.32 0)
 			(hide yes)
 			(show_name no)
@@
 	(symbol
 		(lib_id "Switch:SW_Push")
-		(at 595.63 373.38 0)
+		(at 603.25 373.38 0)
 		(unit 1)
 		(body_style 1)
@@
 		(fields_autoplaced yes)
 		(property "Reference" "SW5"
-			(at 595.63 365.76 0)
+			(at 603.25 365.76 0)
 			(show_name no)
 			(do_not_autoplace no)
@@
 			)
 		)
-		(property "Value" "SW_Push"
-			(at 595.63 368.3 0)
+		(property "Value" "BTN_UP"
+			(at 603.25 368.3 0)
 			(show_name no)
 			(do_not_autoplace no)
@@
 		)
 		(property "Footprint" ""
-			(at 595.63 368.3 0)
+			(at 603.25 368.3 0)
 			(hide yes)
 			(show_name no)
@@
 		)
 		(property "Datasheet" ""
-			(at 595.63 368.3 0)
+			(at 603.25 368.3 0)
 			(hide yes)
 			(show_name no)
@@
 		)
 		(property "Description" "Push button switch, generic, two pins"
-			(at 595.63 373.38 0)
+			(at 603.25 373.38 0)
 			(hide yes)
 			(show_name no)
@@
 	(symbol
 		(lib_id "Switch:SW_Push")
-		(at 566.42 373.38 0)
+		(at 570.23 373.38 0)
 		(unit 1)
 		(body_style 1)
@@
 		(fields_autoplaced yes)
 		(property "Reference" "SW4"
-			(at 566.42 365.76 0)
+			(at 570.23 365.76 0)
 			(show_name no)
 			(do_not_autoplace no)
@@
 			)
 		)
-		(property "Value" "SW_Push"
-			(at 566.42 368.3 0)
+		(property "Value" "BTN_OK"
+			(at 570.23 368.3 0)
 			(show_name no)
 			(do_not_autoplace no)
@@
 		)
 		(property "Footprint" ""
-			(at 566.42 368.3 0)
+			(at 570.23 368.3 0)
 			(hide yes)
 			(show_name no)
@@
 		)
 		(property "Datasheet" ""
-			(at 566.42 368.3 0)
+			(at 570.23 368.3 0)
 			(hide yes)
 			(show_name no)
@@
 		)
 		(property "Description" "Push button switch, generic, two pins"
-			(at 566.42 373.38 0)
+			(at 570.23 373.38 0)
 			(hide yes)
 			(show_name no)

Commit message: lvlvlvlv
Parts:
- added R37, R38, R41, R42, R43, R44: 10R, symbol Device:R
Connections:
- net VDD33: now also R37.2, R38.2, R41.2, R42.2, R43.2, R44.2
- net at SW7.2: now also R43.1
- net at SW8.2: now also R44.1
- net at SW3.2: now also R37.1
- net at SW6.2: now also R42.1
- net at SW5.2: now also R41.1
- net at SW4.2: now also R38.1
Other:
- moved on the sheet: SW3, SW4, SW5, SW6, SW7, SW8

Commit message: un stopable
Connections:
- net GPIO1 is gone; now on net BTN_OK: U1.6 (GPIO1)
- net GPIO2 is gone; now on net BTN_UP: U1.7 (GPIO2)
- net SPICS1 is gone; now on net BTN_POWER: U1.28 (SPICS1)
- net BTN_LEFT: now reaches SW7.1
- net BTN_RIGHT: now reaches SW8.1
- net BTN_POWER: now reaches SW3.1
- net BTN_DOWN: now reaches SW6.1
- net BTN_UP: now reaches SW5.1
- net BTN_OK: now reaches SW4.1

Commit message: bankai
Connections:
- net GPIO15 is gone; now on net BTN_DOWN: U1.21 (XTAL_32K_P)
- net GPIO41 is gone; now on net BTN_LEFT: U1.47 (MTDI)
- net GPIO42: no longer names the net of U1.48 (MTMS)
Changed lines of the file:
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@@
+		)
+	)
+	(global_label "BTN_DOWN"
+		(shape input)
+		(at 83.82 140.97 180)
+		(fields_autoplaced yes)
+		(effects
+			(font
+				(size 1.27 1.27)
+			)
+			(justify right)
+		)
+		(property "Intersheetrefs" "${INTERSHEET_REFS}"
+			(at 70.9167 140.97 0)
+			(hide yes)
+			(show_name no)
+			(do_not_autoplace no)
+			(effects
+				(font
+					(size 1.27 1.27)
+				)
+				(justify right)
+			)
 		)
 	)
@@
 		)
 	)
+	(global_label "BTN_LEFT"
+		(shape input)
+		(at 182.88 130.81 0)
+		(fields_autoplaced yes)
+		(effects
+			(font
+				(size 1.27 1.27)
+			)
+			(justify left)
+		)
+		(property "Intersheetrefs" "${INTERSHEET_REFS}"
+			(at 194.6342 130.81 0)
+			(hide yes)
+			(show_name no)
+			(do_not_autoplace no)
+			(effects
+				(font
+					(size 1.27 1.27)
+				)
+				(justify left)
+			)
+		)
+	)
 	(global_label "SX1276_RESET"
 		(shape input)
@@
 		)
 	)
-	(global_label "GPIO15"
-		(shape input)
-		(at 83.82 140.97 180)
-		(fields_autoplaced yes)
-		(effects
-			(font
-				(size 1.27 1.27)
-			)
-			(justify right)
-		)
-		(property "Intersheetrefs" "${INTERSHEET_REFS}"
-			(at 73.9405 140.97 0)
-			(hide yes)
-			(show_name no)
-			(do_not_autoplace no)
-			(effects
-				(font
-					(size 1.27 1.27)
-				)
-				(justify right)
-			)
-		)
-	)
 	(global_label "CS_PN532"
 		(shape input)
@@
 		)
 	)
-	(global_label "GPIO41"
-		(shape input)
-		(at 182.88 130.81 0)
-		(fields_autoplaced yes)
-		(effects
-			(font
-				(size 1.27 1.27)
-			)
-			(justify left)
-		)
-		(property "Intersheetrefs" "${INTERSHEET_REFS}"
-			(at 192.7595 130.81 0)
-			(hide yes)
-			(show_name no)
-			(do_not_autoplace no)
-			(effects
-				(font
-					(size 1.27 1.27)
-				)
-				(justify left)
-			)
-		)
-	)
 	(global_label "EN_BTN"
 		(shape input)
@@
 			(hide yes)
 			(show_name no)
-			(do_not_autoplace no)
-			(effects
-				(font
-					(size 1.27 1.27)
-				)
-				(justify left)
-			)
-		)
-	)
-	(global_label "GPIO42"
-		(shape input)
-		(at 182.88 133.35 0)
-		(fields_autoplaced yes)
-		(effects
-			(font
-				(size 1.27 1.27)
-			)
-			(justify left)
-		)
-		(property "Intersheetrefs" "${INTERSHEET_REFS}"
-			(at 192.7595 133.35 0)
-			(hide yes)
-			(show_name no)

Commit message: fahh
Connections:
- net BTN_RIGHT: now also U1.48 (MTMS)
Changed lines of the file:
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@@
 	(text "BUTTON"
 		(exclude_from_sim no)
-		(at 562.102 349.758 0)
+		(at 591.82 350.52 0)
 		(effects
 			(font
@@
 	(polyline
 		(pts
-			(xy 574.04 353.06) (xy 574.04 345.44)
+			(xy 603.758 353.822) (xy 603.758 346.202)
 		)
 		(stroke
@@
 	(polyline
 		(pts
-			(xy 551.18 353.06) (xy 574.04 353.06)
+			(xy 580.898 353.822) (xy 603.758 353.822)
 		)
 		(stroke
@@
 	(polyline
 		(pts
-			(xy 551.18 345.44) (xy 551.18 353.06)
+			(xy 580.898 346.202) (xy 580.898 353.822)
 		)
 		(stroke
@@
 		)
 	)
-	(label "GPIO26"
-		(at 152.4 87.63 0)
-		(effects
-			(font
-				(size 1.27 1.27)
-			)
-			(justify left bottom)
-		)
-	)
 	(global_label "SPI_SCK"
 		(shape input)
@@
 			(hide yes)
 			(show_name no)
+			(do_not_autoplace no)
+			(effects
+				(font
+					(size 1.27 1.27)
+				)
+				(justify left)
+			)
+		)
+	)
+	(global_label "BTN_RIGHT"
+		(shape input)
+		(at 182.88 133.35 0)
+		(fields_autoplaced yes)
+		(effects
+			(font
+				(size 1.27 1.27)
+			)
+			(justify left)
+		)
+		(property "Intersheetrefs" "${INTERSHEET_REFS}"
+			(at 195.8438 133.35 0)
+			(hide yes)
+			(show_name no)

Commit message: suiiiiii
Other:
- note added: "Test Points"
Changed lines of the file:
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@@
 		)
 	)
+	(text "Test Points"
+		(exclude_from_sim no)
+		(at 747.268 349.758 0)
+		(effects
+			(font
+				(size 2.54 2.54)
+				(thickness 0.508)
+				(bold yes)
+			)
+		)
+	)
 	(junction
 		(at 436.88 246.38)
@@
 		)
 	)
+	(polyline
+		(pts
+			(xy 822.96 345.44) (xy 822.96 434.34)
+		)
+		(stroke
+			(width 1)
+			(type solid)
+		)
+	)
 	(wire
 		(pts
@@
 	(polyline
 		(pts
+			(xy 731.52 353.06) (xy 764.54 353.06)
+		)
+		(stroke
+			(width 1)
+			(type solid)
+		)
+	)
+	(polyline
+		(pts
 			(xy 208.28 363.22) (xy 304.8 363.22)
 		)
@@
 		)
 	)
+	(polyline
+		(pts
+			(xy 764.54 353.06) (xy 764.54 345.44)
+		)
+		(stroke
+			(width 1)
+			(type solid)
+		)
+	)
 	(wire
 		(pts
@@
 		)
 	)
+	(polyline
+		(pts
+			(xy 822.96 434.34) (xy 670.56 434.34)
+		)
+		(stroke
+			(width 1)
+			(type solid)
+		)
+	)
 	(wire
 		(pts
@@
 	(polyline
 		(pts
+			(xy 731.52 345.44) (xy 731.52 353.06)
+		)
+		(stroke
+			(width 1)
+			(type solid)
+		)
+	)
+	(polyline
+		(pts
 			(xy 322.834 211.582) (xy 322.834 219.202)
 		)
@@
 	(polyline
 		(pts
+			(xy 670.56 345.44) (xy 670.56 434.34)
+		)
+		(stroke
+			(width 1)
+			(type solid)
+		)
+	)
+	(polyline
+		(pts
 			(xy 15.24 345.44) (xy 142.24 345.44)
 		)
@@
 		)
 	)
+	(polyline
+		(pts
+			(xy 670.56 345.44) (xy 822.96 345.44)
+		)
+		(stroke
+			(width 1)
+			(type solid)
+		)
+	)

Commit message: testpoints
Parts:
- added TP1, TP10, TP2, TP3, TP4, TP5, TP6, TP7, TP8, TP9: TestPoint, symbol Connector:TestPoint
