File: flipper black PCB/Flipper black ki cad/.history/Flipper black ki cad.kicad_sch (KiCad schematic)
At the start: 246 parts, among them J1 Barrel_Jack, J2 Value: DISP_3.5_WAVESHARE, P1 JST-2pin, P2 USB_C_Plug_USB2.0, Q1 MMBT2222A, Q2 FS8205A, SW1 SW_Push, SW2 SW_Push, SW3 BTN_POWER, SW4 BTN_OK, SW5 BTN_UP, SW6 BTN_DOWN, SW7 BTN_LEFT, SW8 BTN_RIGHT, U1 ESP32-S3, U10 BGA725L6, U11 TLV70018_SOT23-5, U12 TXB0102DCU, U13 MCP23017x-x-SS, U14 TSOP382xx, U15 TP4056, U17 AP2112K-3.3, U18 DW01A, U2 W25Q128JVS, U3 CC1101, U4 SX1276, U5 PE4259, U6 PE4259, U7 PN5321A3HN, U8 MAX-M8Q, U9 MASW-007221, X1 B3715 868MHz SAW Filter, X2 B3715 868MHz SAW Filter, Y1 40MHz SMD 3225, Y2 26 MHz SMD, Y3 32 MHz SMD, Y4 27.120 MHz

Commit message: yooooo
Parts:
- removed TP6: TestPoint, symbol Connector:TestPoint
- TP1: value TestPoint -> TP_3V3
- TP10: value TestPoint -> TP_RESET
- TP2: value TestPoint -> TP_BAT
- TP3: value TestPoint -> TP_5V
- TP4: value TestPoint -> TP_GND
- TP5: value TestPoint -> TP_BOOT
- TP7: value TestPoint -> TP_IR_TX
Connections:
- net +3V3: now also TP1.1
- net +5V: now also TP3.1
- net GND: now also TP4.1
- net IR_TX: now also TP7.1
- net TP_BAT: now reaches C101.1, P1.1, U15.5 (BAT), U18.5 (VCC)
- net TP_BAT: now also TP2.1
Other:
- moved on the sheet: R34

Commit message: fahhh
Connections:
- net BOOT_BTN: now also TP5.1
- net EN_BTN: now also TP10.1
Changed lines of the file:
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@@
 	(wire
 		(pts
+			(xy 787.4 375.92) (xy 787.4 379.73)
+		)
+		(stroke
+			(width 0)
+			(type default)
+		)
+	)
+	(wire
+		(pts
 			(xy 393.7 256.54) (xy 393.7 259.08)
 		)
@@
 	(wire
 		(pts
+			(xy 685.8 408.94) (xy 685.8 415.29)
+		)
+		(stroke
+			(width 0)
+			(type default)
+		)
+	)
+	(wire
+		(pts
 			(xy 739.14 266.7) (xy 746.76 266.7)
 		)
@@
 		)
 	)
+	(global_label "EN_BTN"
+		(shape input)
+		(at 685.8 415.29 0)
+		(fields_autoplaced yes)
+		(effects
+			(font
+				(size 1.27 1.27)
+			)
+			(justify left)
+		)
+		(property "Intersheetrefs" "${INTERSHEET_REFS}"
+			(at 695.8004 415.29 0)
+			(hide yes)
+			(show_name no)
+			(do_not_autoplace no)
+			(effects
+				(font
+					(size 1.27 1.27)
+				)
+				(justify left)
+			)
+		)
+	)
 	(global_label "GPS_RESET"
 		(shape input)
@@
 			(hide yes)
 			(show_name no)
+			(do_not_autoplace no)
+			(effects
+				(font
+					(size 1.27 1.27)
+				)
+				(justify left)
+			)
+		)
+	)
+	(global_label "BOOT_BTN"
+		(shape input)
+		(at 787.4 379.73 0)
+		(fields_autoplaced yes)
+		(effects
+			(font
+				(size 1.27 1.27)
+			)
+			(justify left)
+		)
+		(property "Intersheetrefs" "${INTERSHEET_REFS}"
+			(at 799.8195 379.73 0)
+			(hide yes)
+			(show_name no)

Commit message: fah
Parts:
- TP8: value TestPoint -> TP_UART_TX
- TP9: value TestPoint -> TP_UART_RX
Connections:
- net TP_UART_TX: now reaches R6.1, U1.49 (U0TXD)
- net TP_UART_TX: now also TP8.1
- net TP_UART_RX: now reaches TP9.1
Other:
- moved on the sheet: R6
Changed lines of the file:
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@@
 	(wire
 		(pts
+			(xy 736.6 408.94) (xy 736.6 415.29)
+		)
+		(stroke
+			(width 0)
+			(type default)
+		)
+	)
+	(wire
+		(pts
 			(xy 74.93 377.19) (xy 82.55 377.19)
 		)
@@
 	(wire
 		(pts
-			(xy 173.99 135.89) (xy 182.88 135.89)
+			(xy 175.26 135.89) (xy 182.88 135.89)
 		)
 		(stroke
@@
 	(wire
 		(pts
-			(xy 151.13 135.89) (xy 166.37 135.89)
+			(xy 151.13 135.89) (xy 167.64 135.89)
 		)
 		(stroke
@@
 	(wire
 		(pts
+			(xy 711.2 408.94) (xy 711.2 415.29)
+		)
+		(stroke
+			(width 0)
+			(type default)
+		)
+	)
+	(wire
+		(pts
 			(xy 204.47 416.56) (xy 204.47 419.1)
 		)
@@
 		)
 	)
+	(global_label "TP_UART_TX"
+		(shape input)
+		(at 151.13 135.89 0)
+		(fields_autoplaced yes)
+		(effects
+			(font
+				(size 1.27 1.27)
+				(thickness 0.254)
+				(bold yes)
+			)
+			(justify left)
+		)
+		(property "Intersheetrefs" "${INTERSHEET_REFS}"
+			(at 165.5978 135.89 0)
+			(hide yes)
+			(show_name no)
+			(do_not_autoplace no)
+			(effects
+				(font
+					(size 1.27 1.27)
+				)
+				(justify left)
+			)
+		)
+	)
 	(global_label "BTN_UP"
 		(shape input)
@@
 			(font
 				(size 1.27 1.27)
-				(thickness 0.254)
-				(bold yes)
+				(thickness 0.1588)
 			)
 			(justify left)
 		)
 		(property "Intersheetrefs" "${INTERSHEET_REFS}"
-			(at 771.9926 379.73 0)
+			(at 771.5166 379.73 0)
 			(hide yes)
 			(show_name no)
@@
 		)
 	)
+	(global_label "TP_UART_RX"
+		(shape input)
+		(at 711.2 415.29 0)
+		(fields_autoplaced yes)
+		(effects
+			(font
+				(size 1.27 1.27)
+				(thickness 0.1588)
+			)
+			(justify left)
+		)
+		(property "Intersheetrefs" "${INTERSHEET_REFS}"
+			(at 725.4942 415.29 0)
+			(hide yes)
+			(show_name no)
+			(do_not_autoplace no)
+			(effects
+				(font
+					(size 1.27 1.27)
+				)
+				(justify left)
+			)
+		)
+	)
 	(global_label "BTN_POWER"
 		(shape input)
@@
 		)
 	)
+	(global_label "TP_UART_TX"
+		(shape input)
+		(at 736.6 415.29 0)
+		(fields_autoplaced yes)
+		(effects
+			(font
+				(size 1.27 1.27)
+				(thickness 0.254)
+				(bold yes)
+			)
+			(justify left)
+		)
+		(property "Intersheetrefs" "${INTERSHEET_REFS}"
+			(at 751.0678 415.29 0)
+			(hide yes)
+			(show_name no)
+			(do_not_autoplace no)
+			(effects
+				(font
+					(size 1.27 1.27)
+				)
+				(justify left)
+			)
+		)
+	)
 	(global_label "RXTX RF sx"
 		(shape input)
@@
 	(symbol
 		(lib_id "Device:R_US")
-		(at 170.18 135.89 90)
+		(at 171.45 135.89 90)
 		(unit 1)
 		(body_style 1)
@@
 		(dnp no)
 		(property "Reference" "R6"
-			(at 165.608 134.874 90)
+			(at 167.894 135.128 90)
 			(show_name no)
 			(do_not_autoplace no)
@@
 		)
 		(property "Value" "499Ohm"
-			(at 176.276 134.62 90)
+			(at 177.8 134.874 90)
 			(show_name no)
 			(do_not_autoplace no)
@@
 		)
 		(property "Footprint" ""
-			(at 170.434 134.874 90)
+			(at 171.704 134.874 90)
 			(hide yes)
 			(show_name no)
@@
 		)
 		(property "Datasheet" ""
-			(at 170.18 135.89 0)
+			(at 171.45 135.89 0)
 			(hide yes)
 			(show_name no)
@@
 		)
 		(property "Description" "Resistor, US symbol"
-			(at 170.18 135.89 0)
+			(at 171.45 135.89 0)
 			(hide yes)
 			(show_name no)
@@
 			)
 		)
-		(property "Value" "TestPoint"
+		(property "Value" "TP_UART_RX"
 			(at 713.74 406.9079 0)
 			(show_name no)
@@
 			)
 		)
-		(property "Value" "TestPoint"
+		(property "Value" "TP_UART_TX"
 			(at 739.14 406.9079 0)
 			(show_name no)

Commit message: more more more
Connections:
- net TP_UART_RX is gone; now on net GPS_RXD: TP9.1

Commit message: lol
Parts:
- added U16: PESD5V0L4UG,115, SOT65P210X110-5N, symbol PESD5V0L4UG_115:PESD5V0L4UG,115
Connections:
- net GND: now also U16.2
- net USB_DN: now also U16.4; no longer P2.A7 (D-)
- net USB_DP: now also U16.5; no longer P2.A6 (D+)
- new net: P2.A6 (D+), U16.1
- new net: P2.A7 (D-), U16.3
Other:
- note added: "D+"
- note added: "D-"
- note added: "ESD Protection"
- moved on the sheet: P2, R40

Commit message: suii
Parts:
- C102, C103: value C -> 10uf
- C14, C25: value 1.0 pF -> 1.0pF
- C26: value 1.5 pf -> 1.5pf
- C27: value 1.5 pF -> 1.5pF
- C91: value C -> 1nf
- C92: value C -> 22pf
- R13: value NC -> 0R
- R26: value R -> 10K
- SW1: value SW_Push -> boot
- SW2: value SW_Push -> REST
Changed lines of the file:
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@@
 			)
 		)
-		(property "Value" "SW_Push"
-			(at 51.308 88.392 0)
+		(property "Value" "boot"
+			(at 49.022 88.392 0)
 			(show_name no)
 			(do_not_autoplace no)
@@
 			)
 		)
-		(property "Value" "1.0 pF"
+		(property "Value" "1.0pF"
 			(at 178.816 284.48 0)
 			(show_name no)
@@
 			)
 		)
-		(property "Value" "C"
+		(property "Value" "22pf"
 			(at 599.186 308.864 90)
 			(show_name no)
@@
 			)
 		)
-		(property "Value" "NC"
+		(property "Value" "0R"
 			(at 499.618 68.072 90)
 			(show_name no)
@@
 			)
 		)
-		(property "Value" "C"
+		(property "Value" "1nf"
 			(at 596.646 299.72 90)
 			(show_name no)
@@
 			)
 		)
-		(property "Value" "SW_Push"
+		(property "Value" "REST"
 			(at 179.07 150.876 0)
 			(show_name no)
@@
 			)
 		)
-		(property "Value" "C"
+		(property "Value" "10uf"
 			(at 379.73 420.3699 0)
 			(show_name no)
@@
 		(in_pos_files yes)
 		(dnp no)
-		(fields_autoplaced yes)
 		(property "Reference" "C26"
-			(at 203.2 271.78 90)
+			(at 202.946 273.558 90)
 			(show_name no)
 			(do_not_autoplace no)
@@
 			)
 		)
-		(property "Value" "1.5 pf"
-			(at 203.2 274.32 90)
+		(property "Value" "1.5pf"
+			(at 202.946 276.098 90)
 			(show_name no)
 			(do_not_autoplace no)
@@
 		(dnp no)
 		(property "Reference" "L11"
-			(at 207.01 286.512 90)
+			(at 207.264 289.052 90)
 			(show_name no)
 			(do_not_autoplace no)
@@
 		)
 		(property "Value" "2.7nH"
-			(at 207.01 288.798 90)
+			(at 212.344 290.068 90)
 			(show_name no)
 			(do_not_autoplace no)
@@
 		(dnp no)
 		(property "Reference" "C27"
-			(at 197.104 285.75 90)
+			(at 196.596 292.1 90)
 			(show_name no)
 			(do_not_autoplace no)
@@
 			)
 		)
-		(property "Value" "1.5 pF"
+		(property "Value" "1.5pF"
 			(at 199.136 287.528 90)
 			(show_name no)
@@
 			)
 		)
-		(property "Value" "R"
-			(at 754.126 265.684 90)
+		(property "Value" "10K"
+			(at 755.396 265.684 90)
 			(show_name no)
 			(do_not_autoplace no)
@@
 			)
 		)
-		(property "Value" "1.0 pF"
+		(property "Value" "1.0pF"
 			(at 185.674 180.086 0)
 			(show_name no)
@@
 			)
 		)
-		(property "Value" "C"
+		(property "Value" "10uf"
 			(at 368.3 421.132 0)
 			(show_name no)

Commit message: sui
Parts:
- C1, C10, C100, C101, C102, C103, C104, C11, C12, C13, C14, C15, C16, C17, C18, C19, C2, C20, C21, C22, C23, C24, C25, C26, C27, C28, C29, C3, C30, C31, C32, C33, C34, C35, C36, C37, C38, C39, C4, C40, C41, C42, C43, C44, C45, C46, C47, C48, C49, C5, C50, C51, C52, C53, C54, C55, C56, C57, C58, C59, C6, C60, C61, C62, C63, C64, C65, C66, C67, C68, C69, C7, C70, C71, C72, C73, C74, C75, C76, C77, C78, C79, C8, C80, C81, C82, C83, C84, C85, C86, C87, C88, C89, C9, C90, C91, C92, C93, C94, C95, C96, C97, C98, C99, C_EN1: footprint (none) -> Capacitor_SMD:C_0603_1608Metric_Pad1.08x0.95mm_HandSolder
- R1, R10, R11, R12, R13, R14, R15, R16, R17, R18, R19, R2, R20, R21, R22, R23, R24, R25, R26, R27, R28, R29, R3, R30, R31, R32, R33, R34, R35, R36, R37, R38, R39, R4, R40, R41, R42, R43, R44, R5, R6, R7, R8, R9, R_BOOT1, R_EN1, R_GPIO45, R_GPIO46, R_I0, R_I1, R_RSTPD1: footprint (none) -> Resistor_SMD:R_0402_1005Metric
- Y1, Y2, Y3, Y4: footprint (none) -> Crystal:Crystal_SMD_2016-4Pin_2.0x1.6mm

Commit message: sui
Other:
- moved on the sheet: C44, C45, L18
Changed lines of the file:
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@@
 	)
 	(junction
-		(at 215.9 279.4)
+		(at 412.75 66.04)
 		(diameter 0)
 		(color 0 0 0 0)
 	)
 	(junction
-		(at 410.21 66.04)
+		(at 215.9 279.4)
 		(diameter 0)
 		(color 0 0 0 0)
@@
 	)
 	(junction
+		(at 391.16 66.04)
+		(diameter 0)
+		(color 0 0 0 0)
+	)
+	(junction
 		(at 62.23 247.65)
 		(diameter 0)
@@
 	)
 	(junction
-		(at 392.43 66.04)
-		(diameter 0)
-		(color 0 0 0 0)
-	)
-	(junction
 		(at 554.99 247.65)
 		(diameter 0)
@@
 	(wire
 		(pts
-			(xy 392.43 66.04) (xy 400.05 66.04)
-		)
-		(stroke
-			(width 0)
-			(type default)
-		)
-	)
-	(wire
-		(pts
 			(xy 739.14 31.75) (xy 739.14 33.02)
 		)
@@
 	(wire
 		(pts
-			(xy 410.21 66.04) (xy 414.02 66.04)
-		)
-		(stroke
-			(width 0)
-			(type default)
-		)
-	)
-	(wire
-		(pts
 			(xy 251.46 400.05) (xy 251.46 398.78)
 		)
@@
 	(wire
 		(pts
-			(xy 421.64 66.04) (xy 429.26 66.04)
+			(xy 424.18 66.04) (xy 429.26 66.04)
 		)
 		(stroke
@@
 	(wire
 		(pts
+			(xy 412.75 66.04) (xy 416.56 66.04)
+		)
+		(stroke
+			(width 0)
+			(type default)
+		)
+	)
+	(wire
+		(pts
 			(xy 303.53 314.96) (xy 316.23 314.96)
 		)
@@
 	(wire
 		(pts
-			(xy 383.54 66.04) (xy 392.43 66.04)
+			(xy 383.54 66.04) (xy 391.16 66.04)
 		)
 		(stroke
@@
 	(wire
 		(pts
-			(xy 407.67 66.04) (xy 410.21 66.04)
+			(xy 407.67 66.04) (xy 412.75 66.04)
 		)
 		(stroke
@@
 	(wire
 		(pts
+			(xy 391.16 66.04) (xy 400.05 66.04)
+		)
+		(stroke
+			(width 0)
+			(type default)
+		)
+	)
+	(wire
+		(pts
 			(xy 87.63 273.05) (xy 111.76 273.05)
 		)
@@
 	(wire
 		(pts
-			(xy 410.21 66.04) (xy 410.21 68.58)
+			(xy 412.75 66.04) (xy 412.75 68.58)
 		)
 		(stroke
@@
 			(font
 				(size 1.27 1.27)
-				(thickness 0.254)
-				(bold yes)
+				(thickness 0.1588)
 			)
 			(justify right)
 		)
 		(property "Intersheetrefs" "${INTERSHEET_REFS}"
-			(at 67.7193 397.51 0)
+			(at 68.1953 397.51 0)
 			(hide yes)
 			(show_name no)
@@
 			(font
 				(size 1.27 1.27)
-				(thickness 0.254)
-				(bold yes)
+				(thickness 0.1588)
 			)
 			(justify left)
 		)
 		(property "Intersheetrefs" "${INTERSHEET_REFS}"
-			(at 51.9631 414.02 0)
+			(at 51.4871 414.02 0)
 			(hide yes)
 			(show_name no)
@@
 			(font
 				(size 1.27 1.27)
-				(thickness 0.254)
-				(bold yes)
+				(thickness 0.1588)
 			)
 			(justify left)
 		)
 		(property "Intersheetrefs" "${INTERSHEET_REFS}"
-			(at 227.1626 398.78 0)
+			(at 226.6866 398.78 0)
 			(hide yes)
 			(show_name no)
@@
 		(dnp no)
 		(property "Reference" "FB1"
-			(at 630.174 284.988 0)
+			(at 633.476 285.75 0)
 			(show_name no)
 			(do_not_autoplace no)
@@
 		(dnp no)
 		(property "Reference" "L19"
-			(at 400.812 63.5 90)
+			(at 400.812 64.516 90)
 			(show_name no)
 			(do_not_autoplace no)
@@
 		)
 		(property "Value" "2.7nH"
-			(at 406.654 63.5 90)
+			(at 406.654 64.516 90)
 			(show_name no)
 			(do_not_autoplace no)
@@
 	(symbol
 		(lib_id "Device:L")
-		(at 392.43 69.85 180)
+		(at 391.16 69.85 180)
 		(unit 1)
 		(body_style 1)
@@
 		(fields_autoplaced yes)
 		(property "Reference" "L18"
-			(at 393.7 68.5799 0)
+			(at 392.43 68.5799 0)
 			(show_name no)
 			(do_not_autoplace no)
@@
 		)
 		(property "Value" "2.7nH"
-			(at 393.7 71.1199 0)
+			(at 392.43 71.1199 0)
 			(show_name no)
 			(do_not_autoplace no)
@@
 		)
 		(property "Footprint" ""
-			(at 392.43 69.85 0)
+			(at 391.16 69.85 0)
 			(hide yes)
 			(show_name no)
@@
 		)
 		(property "Datasheet" ""
-			(at 392.43 69.85 0)
+			(at 391.16 69.85 0)
 			(hide yes)
 			(show_name no)
@@
 		)
 		(property "Description" "Inductor"
-			(at 392.43 69.85 0)
+			(at 391.16 69.85 0)
 			(hide yes)
 			(show_name no)
@@
 		)
 		(property "Field5" ""
-			(at 392.43 69.85 0)
+			(at 391.16 69.85 0)
 			(hide yes)
 			(show_name no)
@@
 	(symbol
 		(lib_id "power:GND")
-		(at 410.21 76.2 0)
+		(at 412.75 76.2 0)
 		(unit 1)
 		(body_style 1)
@@
 		(dnp no)
 		(property "Reference" "#PWR066"
-			(at 410.21 82.55 0)
+			(at 412.75 82.55 0)
 			(hide yes)
 			(show_name no)
@@
 		)
 		(property "Value" "GND"
-			(at 410.21 80.264 0)
+			(at 412.75 80.264 0)
 			(show_name no)
 			(do_not_autoplace no)
@@
 		)
 		(property "Footprint" ""
-			(at 410.21 76.2 0)
+			(at 412.75 76.2 0)
 			(hide yes)
 			(show_name no)
@@
 		)
 		(property "Datasheet" ""
-			(at 410.21 76.2 0)
+			(at 412.75 76.2 0)
 			(hide yes)
 			(show_name no)
@@
 		)
 		(property "Description" "Power symbol creates a global label with name \"GND\" , ground"
-			(at 410.21 76.2 0)
+			(at 412.75 76.2 0)
 			(hide yes)
 			(show_name no)
@@
 	(symbol
 		(lib_id "Device:C")
-		(at 417.83 66.04 90)
+		(at 420.37 66.04 90)
 		(unit 1)
 		(body_style 1)
@@
 		(dnp no)
 		(property "Reference" "C45"
-			(at 415.544 61.976 90)
+			(at 418.084 61.976 90)
 			(show_name no)
 			(do_not_autoplace no)
@@
 		)
 		(property "Value" "3.3pf"
-			(at 420.878 62.738 90)
+			(at 423.418 62.738 90)
 			(show_name no)
 			(do_not_autoplace no)
@@
 		)
 		(property "Footprint" "Capacitor_SMD:C_0603_1608Metric_Pad1.08x0.95mm_HandSolder"
-			(at 421.64 65.0748 0)
+			(at 424.18 65.0748 0)
 			(hide yes)
 			(show_name no)
@@
 		)
 		(property "Datasheet" ""
-			(at 417.83 66.04 0)
+			(at 420.37 66.04 0)
 			(hide yes)
 			(show_name no)
@@
 		)
 		(property "Description" "Unpolarized capacitor"
-			(at 417.83 66.04 0)
+			(at 420.37 66.04 0)
 			(hide yes)
 			(show_name no)
@@
 	(symbol
 		(lib_id "power:GND")
-		(at 392.43 73.66 0)
+		(at 391.16 73.66 0)
 		(unit 1)
 		(body_style 1)
@@
 		(dnp no)
 		(property "Reference" "#PWR065"
-			(at 392.43 80.01 0)
+			(at 391.16 80.01 0)
 			(hide yes)
 			(show_name no)
@@
 		)
 		(property "Value" "GND"
-			(at 392.176 77.724 0)
+			(at 390.906 77.724 0)
 			(show_name no)
 			(do_not_autoplace no)
@@
 		)
 		(property "Footprint" ""
-			(at 392.43 73.66 0)
+			(at 391.16 73.66 0)
 			(hide yes)
 			(show_name no)
@@
 		)
 		(property "Datasheet" ""
-			(at 392.43 73.66 0)
+			(at 391.16 73.66 0)
 			(hide yes)
 			(show_name no)
@@
 		)
 		(property "Description" "Power symbol creates a global label with name \"GND\" , ground"
-			(at 392.43 73.66 0)
+			(at 391.16 73.66 0)
 			(hide yes)
 			(show_name no)
@@
 	(symbol
 		(lib_id "Device:C")
-		(at 410.21 72.39 0)
+		(at 412.75 72.39 0)
 		(unit 1)
 		(body_style 1)
@@
 		(in_pos_files yes)
 		(dnp no)
-		(fields_autoplaced yes)
 		(property "Reference" "C44"
-			(at 414.02 71.1199 0)
+			(at 415.29 72.39 0)
 			(show_name no)
 			(do_not_autoplace no)
@@
 		)
 		(property "Value" "3.3pf"
-			(at 414.02 73.6599 0)
+			(at 415.036 74.422 0)
 			(show_name no)
 			(do_not_autoplace no)
@@
 		)
 		(property "Footprint" "Capacitor_SMD:C_0603_1608Metric_Pad1.08x0.95mm_HandSolder"
-			(at 411.1752 76.2 0)
+			(at 413.7152 76.2 0)
 			(hide yes)
 			(show_name no)
@@
 		)
 		(property "Datasheet" ""
-			(at 410.21 72.39 0)
+			(at 412.75 72.39 0)
 			(hide yes)
 			(show_name no)
@@
 		)
 		(property "Description" "Unpolarized capacitor"
-			(at 410.21 72.39 0)
+			(at 412.75 72.39 0)
 			(hide yes)
 			(show_name no)
