File: flipper black PCB/Flipper black ki cad/.history/Flipper black ki cad.kicad_sch (KiCad schematic)
At the start: 246 parts, among them J1 Barrel_Jack, J2 Value: DISP_3.5_WAVESHARE, P1 JST-2pin, P2 USB_C_Plug_USB2.0, Q1 MMBT2222A, Q2 FS8205A, SW1 boot, SW2 REST, SW3 BTN_POWER, SW4 BTN_OK, SW5 BTN_UP, SW6 BTN_DOWN, SW7 BTN_LEFT, SW8 BTN_RIGHT, U1 ESP32-S3, U10 BGA725L6, U11 TLV70018_SOT23-5, U12 TXB0102DCU, U13 MCP23017x-x-SS, U14 TSOP382xx, U15 TP4056, U16 PESD5V0L4UG,115, U17 AP2112K-3.3, U18 DW01A, U2 W25Q128JVS, U3 CC1101, U4 SX1276, U5 PE4259, U6 PE4259, U7 PN5321A3HN, U8 MAX-M8Q, U9 MASW-007221, X1 433MHz SAW Filter, X2 B3715 868MHz SAW Filter, Y1 40MHz SMD 3225, Y2 26 MHz SMD, Y3 32 MHz SMD, Y4 27.120 MHz

Commit message: uo
Parts:
- added C105: 100pf, symbol Device:C
Connections:
- net GND: now also C105.2
- net at L27.2, U10.5 (AI): now also C105.1
Other:
- moved on the sheet: GPS_ANT1, L27
Changed lines of the file:
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@@
 	)
 	(junction
+		(at 712.47 309.88)
+		(diameter 0)
+		(color 0 0 0 0)
+	)
+	(junction
 		(at 119.38 59.69)
 		(diameter 0)
@@
 	(wire
 		(pts
-			(xy 708.66 307.34) (xy 708.66 309.88)
+			(xy 712.47 307.34) (xy 712.47 309.88)
 		)
 		(stroke
@@
 	(wire
 		(pts
-			(xy 708.66 294.64) (xy 708.66 299.72)
+			(xy 712.47 294.64) (xy 712.47 299.72)
 		)
 		(stroke
@@
 	(wire
 		(pts
-			(xy 694.69 309.88) (xy 708.66 309.88)
+			(xy 694.69 309.88) (xy 712.47 309.88)
 		)
 		(stroke
@@
 	(symbol
 		(lib_id "Device:Antenna")
-		(at 708.66 289.56 0)
+		(at 712.47 289.56 0)
 		(unit 1)
 		(body_style 1)
@@
 		(in_pos_files yes)
 		(dnp no)
-		(fields_autoplaced yes)
 		(property "Reference" "GPS_ANT1"
-			(at 711.2 288.9249 0)
+			(at 708.914 282.956 0)
 			(show_name no)
 			(do_not_autoplace no)
@@
 		)
 		(property "Value" "50ohm"
-			(at 711.2 291.4649 0)
+			(at 708.914 285.496 0)
 			(show_name no)
 			(do_not_autoplace no)
@@
 		)
 		(property "Footprint" "Connector_Coaxial:U.FL_Hirose_U.FL-R-SMT-1_Vertical"
-			(at 708.66 289.56 0)
+			(at 712.47 289.56 0)
 			(hide yes)
 			(show_name no)
@@
 		)
 		(property "Datasheet" ""
-			(at 708.66 289.56 0)
+			(at 712.47 289.56 0)
 			(hide yes)
 			(show_name no)
@@
 		)
 		(property "Description" "Antenna"
-			(at 708.66 289.56 0)
+			(at 712.47 289.56 0)
 			(hide yes)
 			(show_name no)
@@
 	(symbol
 		(lib_id "Device:L")
-		(at 708.66 303.53 0)
+		(at 712.47 303.53 0)
 		(unit 1)
 		(body_style 1)
@@
 		(in_pos_files yes)
 		(dnp no)
-		(fields_autoplaced yes)
 		(property "Reference" "L27"
-			(at 709.93 302.2599 0)
+			(at 712.47 299.974 0)
 			(show_name no)
 			(do_not_autoplace no)
@@
 		)
 		(property "Value" "5.6nH"
-			(at 709.93 304.7999 0)
+			(at 713.74 302.006 0)
 			(show_name no)
 			(do_not_autoplace no)
@@
 		)
 		(property "Footprint" "Inductor_SMD:L_0603_1608Metric_Pad1.05x0.95mm_HandSolder"
-			(at 708.66 303.53 0)
+			(at 712.47 303.53 0)
 			(hide yes)
 			(show_name no)
@@
 		)
 		(property "Datasheet" ""
-			(at 708.66 303.53 0)
+			(at 712.47 303.53 0)
 			(hide yes)
 			(show_name no)
@@
 		)
 		(property "Description" "Inductor"
-			(at 708.66 303.53 0)
+			(at 712.47 303.53 0)
 			(hide yes)
 			(show_name no)
@@
 	(symbol
 		(lib_id "power:GND")
+		(at 712.47 317.5 0)
+		(unit 1)
+		(body_style 1)
+		(exclude_from_sim no)
+		(in_bom yes)
+		(on_board yes)
+		(in_pos_files yes)
+		(dnp no)
+		(property "Reference" "#PWR0186"
+			(at 712.47 323.85 0)
+			(hide yes)
+			(show_name no)
+			(do_not_autoplace no)
+			(effects
+				(font
+					(size 1.27 1.27)
+				)
+			)
+		)
+		(property "Value" "GND"
+			(at 712.47 321.056 0)
+			(show_name no)
+			(do_not_autoplace no)
+			(effects
+				(font
+					(size 1.27 1.27)
+				)
+			)
+		)
+		(property "Footprint" ""
+			(at 712.47 317.5 0)
+			(hide yes)
+			(show_name no)
+			(do_not_autoplace no)
+			(effects
+				(font
+					(size 1.27 1.27)
+				)
+			)
+		)
+		(property "Datasheet" ""
+			(at 712.47 317.5 0)
+			(hide yes)
+			(show_name no)
+			(do_not_autoplace no)
+			(effects
+				(font
+					(size 1.27 1.27)
+				)
+			)
+		)
+		(property "Description" "Power symbol creates a global label with name \"GND\" , ground"
+			(at 712.47 317.5 0)
+			(hide yes)
+			(show_name no)
+			(do_not_autoplace no)
+			(effects
+				(font
+					(size 1.27 1.27)
+				)
+			)
+		)
+		(pin "1"
+		)
+		(instances
+			(project "Flipper black ki cad"
+				(path "/aadf5baa-c41c-48f9-af5f-e274c89cf282"
+					(reference "#PWR0186")
+					(unit 1)
+				)
+			)
+		)
+	)
+	(symbol
+		(lib_id "power:GND")
 		(at 444.5 76.2 0)
 		(unit 1)
@@
 					(unit 1)
 				)
+			)
+		)
+	)
+	(symbol
+		(lib_id "Device:C")
+		(at 712.47 313.69 0)
+		(unit 1)
+		(body_style 1)
+		(exclude_from_sim no)
+		(in_bom yes)
+		(on_board yes)
+		(in_pos_files yes)
+		(dnp no)
+		(property "Reference" "C105"
+			(at 715.518 312.42 0)
+			(show_name no)
+			(do_not_autoplace no)
+			(effects
+				(font
+					(size 1.27 1.27)
+				)
+				(justify left)
+			)
+		)
+		(property "Value" "100pf"
+			(at 715.518 314.96 0)
+			(show_name no)
+			(do_not_autoplace no)
+			(effects
+				(font
+					(size 1.27 1.27)
+				)
+				(justify left)
+			)
+		)
+		(property "Footprint" ""
+			(at 713.4352 317.5 0)
+			(hide yes)
+			(show_name no)
+			(do_not_autoplace no)
+			(effects
+				(font
+					(size 1.27 1.27)
+				)
+			)
+		)
+		(property "Datasheet" ""
+			(at 712.47 313.69 0)
+			(hide yes)
+			(show_name no)
+			(do_not_autoplace no)
+			(effects
+				(font
+					(size 1.27 1.27)
+				)
+			)
+		)
+		(property "Description" "Unpolarized capacitor"
+			(at 712.47 313.69 0)
+			(hide yes)
+			(show_name no)
+			(do_not_autoplace no)
+			(effects
+				(font
+					(size 1.27 1.27)
+				)
+			)
+		)
+		(pin "2"
+		)
+		(pin "1"
+		)
+		(instances
+			(project "Flipper black ki cad"
+				(path "/aadf5baa-c41c-48f9-af5f-e274c89cf282"
+					(reference "C105")
+					(unit 1)
+				)

Commit message: yeee
Connections:
- net GND: no longer C105.2
- net at C105.1, L27.2: no longer U10.5 (AI)
- new net: C105.2, U10.5 (AI)
Other:
- moved on the sheet: GPS_ANT1, L27
Changed lines of the file:
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@@
 	)
 	(junction
-		(at 712.47 309.88)
-		(diameter 0)
-		(color 0 0 0 0)
-	)
-	(junction
 		(at 119.38 59.69)
 		(diameter 0)
@@
 	(wire
 		(pts
-			(xy 712.47 307.34) (xy 712.47 309.88)
+			(xy 712.47 294.64) (xy 712.47 297.18)
 		)
 		(stroke
@@
 	(wire
 		(pts
-			(xy 712.47 294.64) (xy 712.47 299.72)
+			(xy 712.47 281.94) (xy 712.47 287.02)
 		)
 		(stroke
@@
 		)
 	)
+	(wire
+		(pts
+			(xy 712.47 304.8) (xy 712.47 309.88)
+		)
+		(stroke
+			(width 0)
+			(type default)
+		)
+	)
 	(polyline
 		(pts
@@
 	(symbol
 		(lib_id "Device:Antenna")
-		(at 712.47 289.56 0)
+		(at 712.47 276.86 0)
 		(unit 1)
 		(body_style 1)
@@
 		(dnp no)
 		(property "Reference" "GPS_ANT1"
-			(at 708.914 282.956 0)
+			(at 708.914 270.256 0)
 			(show_name no)
 			(do_not_autoplace no)
@@
 		)
 		(property "Value" "50ohm"
-			(at 708.914 285.496 0)
+			(at 708.914 272.796 0)
 			(show_name no)
 			(do_not_autoplace no)
@@
 		)
 		(property "Footprint" "Connector_Coaxial:U.FL_Hirose_U.FL-R-SMT-1_Vertical"
-			(at 712.47 289.56 0)
+			(at 712.47 276.86 0)
 			(hide yes)
 			(show_name no)
@@
 		)
 		(property "Datasheet" ""
-			(at 712.47 289.56 0)
+			(at 712.47 276.86 0)
 			(hide yes)
 			(show_name no)
@@
 		)
 		(property "Description" "Antenna"
-			(at 712.47 289.56 0)
+			(at 712.47 276.86 0)
 			(hide yes)
 			(show_name no)
@@
 	(symbol
 		(lib_id "Device:L")
-		(at 712.47 303.53 0)
+		(at 712.47 290.83 0)
 		(unit 1)
 		(body_style 1)
@@
 		(dnp no)
 		(property "Reference" "L27"
-			(at 712.47 299.974 0)
+			(at 712.47 287.274 0)
 			(show_name no)
 			(do_not_autoplace no)
@@
 		)
 		(property "Value" "5.6nH"
-			(at 713.74 302.006 0)
+			(at 713.74 289.306 0)
 			(show_name no)
 			(do_not_autoplace no)
@@
 		)
 		(property "Footprint" "Inductor_SMD:L_0603_1608Metric_Pad1.05x0.95mm_HandSolder"
-			(at 712.47 303.53 0)
+			(at 712.47 290.83 0)
 			(hide yes)
 			(show_name no)
@@
 		)
 		(property "Datasheet" ""
-			(at 712.47 303.53 0)
+			(at 712.47 290.83 0)
 			(hide yes)
 			(show_name no)
@@
 		)
 		(property "Description" "Inductor"
-			(at 712.47 303.53 0)
+			(at 712.47 290.83 0)
 			(hide yes)
 			(show_name no)
@@
 	(symbol
 		(lib_id "power:GND")
-		(at 712.47 317.5 0)
-		(unit 1)
-		(body_style 1)
-		(exclude_from_sim no)
-		(in_bom yes)
-		(on_board yes)
-		(in_pos_files yes)
-		(dnp no)
-		(property "Reference" "#PWR0186"
-			(at 712.47 323.85 0)
-			(hide yes)
-			(show_name no)
-			(do_not_autoplace no)
-			(effects
-				(font
-					(size 1.27 1.27)
-				)
-			)
-		)
-		(property "Value" "GND"
-			(at 712.47 321.056 0)
-			(show_name no)
-			(do_not_autoplace no)
-			(effects
-				(font
-					(size 1.27 1.27)
-				)
-			)
-		)
-		(property "Footprint" ""
-			(at 712.47 317.5 0)
-			(hide yes)
-			(show_name no)
-			(do_not_autoplace no)
-			(effects
-				(font
-					(size 1.27 1.27)
-				)
-			)
-		)
-		(property "Datasheet" ""
-			(at 712.47 317.5 0)
-			(hide yes)
-			(show_name no)
-			(do_not_autoplace no)
-			(effects
-				(font
-					(size 1.27 1.27)
-				)
-			)
-		)
-		(property "Description" "Power symbol creates a global label with name \"GND\" , ground"
-			(at 712.47 317.5 0)
-			(hide yes)
-			(show_name no)
-			(do_not_autoplace no)
-			(effects
-				(font
-					(size 1.27 1.27)
-				)
-			)
-		)
-		(pin "1"
-		)
-		(instances
-			(project "Flipper black ki cad"
-				(path "/aadf5baa-c41c-48f9-af5f-e274c89cf282"
-					(reference "#PWR0186")
-					(unit 1)
-				)
-			)
-		)
-	)
-	(symbol
-		(lib_id "power:GND")
 		(at 444.5 76.2 0)
 		(unit 1)
@@
 	)
 	(symbol
+		(lib_id "Device:C")
+		(at 712.47 300.99 0)
+		(unit 1)
+		(body_style 1)
+		(exclude_from_sim no)
+		(in_bom yes)
+		(on_board yes)
+		(in_pos_files yes)
+		(dnp no)
+		(property "Reference" "C105"
+			(at 715.518 299.72 0)
+			(show_name no)
+			(do_not_autoplace no)
+			(effects
+				(font
+					(size 1.27 1.27)
+				)
+				(justify left)
+			)
+		)
+		(property "Value" "100pf"
+			(at 715.518 302.26 0)
+			(show_name no)
+			(do_not_autoplace no)
+			(effects
+				(font
+					(size 1.27 1.27)
+				)
+				(justify left)
+			)
+		)
+		(property "Footprint" ""
+			(at 713.4352 304.8 0)
+			(hide yes)
+			(show_name no)
+			(do_not_autoplace no)
+			(effects
+				(font
+					(size 1.27 1.27)
+				)
+			)
+		)
+		(property "Datasheet" ""
+			(at 712.47 300.99 0)
+			(hide yes)
+			(show_name no)
+			(do_not_autoplace no)
+			(effects
+				(font
+					(size 1.27 1.27)
+				)
+			)
+		)
+		(property "Description" "Unpolarized capacitor"
+			(at 712.47 300.99 0)
+			(hide yes)
+			(show_name no)
+			(do_not_autoplace no)
+			(effects
+				(font
+					(size 1.27 1.27)
+				)
+			)
+		)
+		(pin "2"
+		)
+		(pin "1"
+		)
+		(instances
+			(project "Flipper black ki cad"
+				(path "/aadf5baa-c41c-48f9-af5f-e274c89cf282"
+					(reference "C105")
+					(unit 1)
+				)
+			)
+		)
+	)
+	(symbol
 		(lib_id "RF_NFC:PN5321A3HN_C1xx")
 		(at 336.55 292.1 0)
@@
 					(unit 1)
 				)
-			)
-		)
-	)
-	(symbol
-		(lib_id "Device:C")
-		(at 712.47 313.69 0)
-		(unit 1)
-		(body_style 1)
-		(exclude_from_sim no)
-		(in_bom yes)
-		(on_board yes)
-		(in_pos_files yes)
-		(dnp no)
-		(property "Reference" "C105"
-			(at 715.518 312.42 0)
-			(show_name no)
-			(do_not_autoplace no)
-			(effects
-				(font
-					(size 1.27 1.27)
-				)
-				(justify left)
-			)
-		)
-		(property "Value" "100pf"
-			(at 715.518 314.96 0)
-			(show_name no)
-			(do_not_autoplace no)
-			(effects
-				(font
-					(size 1.27 1.27)
-				)
-				(justify left)
-			)
-		)
-		(property "Footprint" ""
-			(at 713.4352 317.5 0)
-			(hide yes)
-			(show_name no)
-			(do_not_autoplace no)
-			(effects
-				(font
-					(size 1.27 1.27)
-				)
-			)
-		)
-		(property "Datasheet" ""
-			(at 712.47 313.69 0)
-			(hide yes)
-			(show_name no)
-			(do_not_autoplace no)
-			(effects
-				(font
-					(size 1.27 1.27)
-				)
-			)
-		)
-		(property "Description" "Unpolarized capacitor"
-			(at 712.47 313.69 0)
-			(hide yes)
-			(show_name no)
-			(do_not_autoplace no)
-			(effects
-				(font
-					(size 1.27 1.27)
-				)
-			)
-		)
-		(pin "2"
-		)
-		(pin "1"
-		)
-		(instances
-			(project "Flipper black ki cad"
-				(path "/aadf5baa-c41c-48f9-af5f-e274c89cf282"
-					(reference "C105")
-					(unit 1)
-				)

Commit message: yooohhohoh
Parts:
- removed J1: Barrel_Jack, Connector_BarrelJack:BarrelJack_Wuerth_694108106102_2.5x5.5mm, symbol Connector:Barrel_Jack
Connections:
- net at FB1.2: now also C91.2
Changed lines of the file:
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@@
 	(wire
 		(pts
-			(xy 628.65 300.99) (xy 613.41 300.99)
-		)
-		(stroke
-			(width 0)
-			(type default)
-		)
-	)
-	(wire
-		(pts
 			(xy 393.7 234.95) (xy 401.32 234.95)
 		)
@@
 	(wire
 		(pts
-			(xy 603.25 300.99) (xy 608.33 300.99)
+			(xy 603.25 300.99) (xy 628.65 300.99)
 		)
 		(stroke
@@
 					(unit 1)
 				)
-			)
-		)
-	)
-	(symbol
-		(lib_id "Connector:Barrel_Jack")
-		(at 610.87 293.37 270)
-		(unit 1)
-		(body_style 1)
-		(exclude_from_sim no)
-		(in_bom yes)
-		(on_board yes)
-		(in_pos_files yes)
-		(dnp no)
-		(fields_autoplaced yes)
-		(property "Reference" "J1"
-			(at 615.95 292.0999 90)
-			(show_name no)
-			(do_not_autoplace no)
-			(effects
-				(font
-					(size 1.27 1.27)
-				)
-				(justify left)
-			)
-		)
-		(property "Value" "Barrel_Jack"
-			(at 615.95 294.6399 90)
-			(show_name no)
-			(do_not_autoplace no)
-			(effects
-				(font
-					(size 1.27 1.27)
-				)
-				(justify left)
-			)
-		)
-		(property "Footprint" "Connector_BarrelJack:BarrelJack_Wuerth_694108106102_2.5x5.5mm"
-			(at 609.854 294.64 0)
-			(hide yes)
-			(show_name no)
-			(do_not_autoplace no)
-			(effects
-				(font
-					(size 1.27 1.27)
-				)
-			)
-		)
-		(property "Datasheet" ""
-			(at 609.854 294.64 0)
-			(hide yes)
-			(show_name no)
-			(do_not_autoplace no)
-			(effects
-				(font
-					(size 1.27 1.27)
-				)
-			)
-		)
-		(property "Description" "DC Barrel Jack"
-			(at 610.87 293.37 0)
-			(hide yes)
-			(show_name no)
-			(do_not_autoplace no)
-			(effects
-				(font
-					(size 1.27 1.27)
-				)
-			)
-		)
-		(pin "1"
-		)
-		(pin "2"
-		)
-		(instances
-			(project "Flipper black ki cad"
-				(path "/aadf5baa-c41c-48f9-af5f-e274c89cf282"
-					(reference "J1")
-					(unit 1)
-				)

Commit message: ahhh
Parts:
- L13, L14, L24: value 2.7nH -> 100nH
- L15, L16, L17, L20: value 2.7nH -> 120nH
- L18, L19: value 2.7nH -> 68nH
- L21, L22, L23: value 2.7nH -> 22nH
Changed lines of the file:
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@@
 			)
 		)
-		(property "Value" "2.7nH"
+		(property "Value" "100nH"
 			(at 400.05 96.52 90)
 			(show_name no)
@@
 			)
 		)
-		(property "Value" "2.7nH"
+		(property "Value" "22nH"
 			(at 508 136.652 90)
 			(show_name no)
@@
 			)
 		)
-		(property "Value" "2.7nH"
+		(property "Value" "68nH"
 			(at 406.654 64.516 90)
 			(show_name no)
@@
 			)
 		)
-		(property "Value" "2.7nH"
+		(property "Value" "100nH"
 			(at 408.94 110.4899 0)
 			(show_name no)
@@
 			)
 		)
-		(property "Value" "2.7nH"
+		(property "Value" "120nH"
 			(at 464.058 97.282 90)
 			(show_name no)
@@
 			)
 		)
-		(property "Value" "2.7nH"
+		(property "Value" "120nH"
 			(at 608.838 70.612 90)
 			(show_name no)
@@
 			)
 		)
-		(property "Value" "2.7nH"
+		(property "Value" "22nH"
 			(at 489.458 137.414 90)
 			(show_name no)
@@
 			)
 		)
-		(property "Value" "2.7nH"
+		(property "Value" "68nH"
 			(at 392.43 71.1199 0)
 			(show_name no)
@@
 			)
 		)
-		(property "Value" "2.7nH"
+		(property "Value" "120nH"
 			(at 481.838 97.282 90)
 			(show_name no)
@@
 		(dnp no)
 		(property "Reference" "C45"
-			(at 418.084 61.976 90)
+			(at 417.068 64.516 90)
 			(show_name no)
 			(do_not_autoplace no)
@@
 		)
 		(property "Value" "3.3pf"
-			(at 423.418 62.738 90)
+			(at 423.926 64.516 90)
 			(show_name no)
 			(do_not_autoplace no)
@@
 			)
 		)
-		(property "Value" "2.7nH"
+		(property "Value" "120nH"
 			(at 446.278 97.282 90)
 			(show_name no)
@@
 			)
 		)
-		(property "Value" "2.7nH"
+		(property "Value" "22nH"
 			(at 450.85 179.07 90)
 			(show_name no)
@@
 			)
 		)
-		(property "Value" "2.7nH"
-			(at 622.808 164.338 90)
+		(property "Value" "100nH"
+			(at 623.062 163.83 90)
 			(show_name no)
 			(do_not_autoplace no)

Commit message: agg aggg
Parts:
- L10, L9: value 2.7nH -> 47nH
- L5, L6, L7, L8: value 2.7nH -> 27nH
Connections:
- net 12C_SDA: now also U13.13 (SDA)
- net GPS_RXD: no longer TP9.1
- net I2C_SDA: no longer U13.13 (SDA)
- net TOUCH_IRQ: no longer U13.28 (GPA7)
- net TOUCH_RST: now also U13.28 (GPA7)
- net TP_UART_TX: no longer R6.1, U1.49 (U0TXD)
- new net: R6.1, U1.49 (U0TXD)
- new net TP_UART_RX: TP9.1
- no-connect marks 13 -> 20
Changed lines of the file:
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@@
 	)
 	(no_connect
+		(at 331.47 128.27)
+	)
+	(no_connect
+		(at 182.88 100.33)
+	)
+	(no_connect
+		(at 331.47 125.73)
+	)
+	(no_connect
+		(at 331.47 133.35)
+	)
+	(no_connect
 		(at 356.87 287.02)
 	)
@@
 	)
 	(no_connect
+		(at 331.47 130.81)
+	)
+	(no_connect
 		(at 356.87 289.56)
 	)
 	(no_connect
+		(at 182.88 102.87)
+	)
+	(no_connect
 		(at 316.23 271.78)
 	)
@@
 	)
 	(no_connect
+		(at 331.47 123.19)
+	)
+	(no_connect
 		(at 316.23 294.64)
 	)
@@
 	(wire
 		(pts
-			(xy 151.13 138.43) (xy 182.88 138.43)
-		)
-		(stroke
-			(width 0)
-			(type default)
-		)
-	)
-	(wire
-		(pts
 			(xy 431.8 416.56) (xy 431.8 412.75)
 		)
@@
 	(wire
 		(pts
-			(xy 284.48 386.08) (xy 264.16 386.08)
+			(xy 284.48 386.08) (xy 271.78 386.08)
 		)
 		(stroke
@@
 	(wire
 		(pts
+			(xy 151.13 138.43) (xy 182.88 138.43)
+		)
+		(stroke
+			(width 0)
+			(type default)
+		)
+	)
+	(wire
+		(pts
 			(xy 251.46 410.21) (xy 251.46 420.37)
 		)
@@
 	(wire
 		(pts
-			(xy 264.16 386.08) (xy 264.16 381)
+			(xy 271.78 386.08) (xy 271.78 381)
 		)
 		(stroke
@@
 	(wire
 		(pts
-			(xy 264.16 381) (xy 272.796 381)
+			(xy 271.78 381) (xy 272.796 381)
 		)
 		(stroke
@@
 		)
 	)
-	(global_label "TP_UART_TX"
-		(shape input)
-		(at 151.13 135.89 0)
-		(fields_autoplaced yes)
-		(effects
-			(font
-				(size 1.27 1.27)
-				(thickness 0.1588)
-			)
-			(justify left)
-		)
-		(property "Intersheetrefs" "${INTERSHEET_REFS}"
-			(at 165.1218 135.89 0)
-			(hide yes)
-			(show_name no)
-			(do_not_autoplace no)
-			(effects
-				(font
-					(size 1.27 1.27)
-				)
-				(justify left)
-			)
-		)
-	)
 	(global_label "BTN_UP"
 		(shape input)
@@
 		)
 	)
-	(global_label "I2C_SDA"
-		(shape input)
-		(at 774.7 120.65 180)
-		(fields_autoplaced yes)
-		(effects
-			(font
-				(size 1.27 1.27)
-			)
-			(justify right)
-		)
-		(property "Intersheetrefs" "${INTERSHEET_REFS}"
-			(at 764.0948 120.65 0)
-			(hide yes)
-			(show_name no)
-			(do_not_autoplace no)
-			(effects
-				(font
-					(size 1.27 1.27)
-				)
-				(justify right)
-			)
-		)
-	)
 	(global_label "DISP_BL"
 		(shape input)
@@
 		)
 	)
-	(global_label "TP_UART_RX"
-		(shape input)
-		(at 151.13 138.43 0)
-		(fields_autoplaced yes)
-		(effects
-			(font
-				(size 1.27 1.27)
-				(thickness 0.1588)
-			)
-			(justify left)
-		)
-		(property "Intersheetrefs" "${INTERSHEET_REFS}"
-			(at 165.4242 138.43 0)
-			(hide yes)
-			(show_name no)
-			(do_not_autoplace no)
-			(effects
-				(font
-					(size 1.27 1.27)
-				)
-				(justify left)
-			)
-		)
-	)
 	(global_label "BTN_POWER"
 		(shape input)
@@
 		)
 	)
-	(global_label "TOUCH_IRQ"
+	(global_label "GPS_EXTINT"
 		(shape input)
-		(at 800.1 135.89 0)
+		(at 510.54 300.99 180)
 		(fields_autoplaced yes)
 		(effects
@@
 				(thickness 0.1588)
 			)
-			(justify left)
+			(justify right)
 		)
 		(property "Intersheetrefs" "${INTERSHEET_REFS}"
-			(at 813.4872 135.89 0)
+			(at 496.6087 300.99 0)
 			(hide yes)
 			(show_name no)
@@
 					(size 1.27 1.27)
 				)
-				(justify left)
+				(justify right)
 			)
 		)
 	)
-	(global_label "GPS_EXTINT"
+	(global_label "CS_SX1276"
 		(shape input)
-		(at 510.54 300.99 180)
+		(at 182.88 110.49 0)
 		(fields_autoplaced yes)
 		(effects
@@
 				(thickness 0.1588)
 			)
-			(justify right)
+			(justify left)
 		)
 		(property "Intersheetrefs" "${INTERSHEET_REFS}"
-			(at 496.6087 300.99 0)
+			(at 196.5693 110.49 0)
 			(hide yes)
 			(show_name no)
@@
 					(size 1.27 1.27)
 				)
-				(justify right)
+				(justify left)
 			)
 		)
 	)
-	(global_label "CS_SX1276"
+	(global_label "TOUCH_RST"
 		(shape input)
-		(at 182.88 110.49 0)
+		(at 800.1 135.89 0)
 		(fields_autoplaced yes)
 		(effects
@@
 		)
 		(property "Intersheetrefs" "${INTERSHEET_REFS}"
-			(at 196.5693 110.49 0)
+			(at 813.729 135.89 0)
 			(hide yes)
 			(show_name no)
@@
 		)
 	)
+	(global_label "12C_SDA"
+		(shape input)
+		(at 774.7 120.65 180)
+		(fields_autoplaced yes)
+		(effects
+			(font
+				(size 1.27 1.27)
+				(thickness 0.1588)
+			)
+			(justify right)
+		)
+		(property "Intersheetrefs" "${INTERSHEET_REFS}"
+			(at 763.4901 120.65 0)
+			(hide yes)
+			(show_name no)
+			(do_not_autoplace no)
+			(effects
+				(font
+					(size 1.27 1.27)
+				)
+				(justify right)
+			)
+		)
+	)
 	(global_label "IR_TX"
 		(shape input)
@@
 			)
 		)
-		(property "Value" "2.7nH"
+		(property "Value" "47nH"
 			(at 181.61 277.368 90)
 			(show_name no)
@@
 			)
 		)
-		(property "Value" "2.7nH"
+		(property "Value" "27nH"
 			(at 130.81 283.718 90)
 			(show_name no)
@@
 			)
 		)
-		(property "Value" "2.7nH"
+		(property "Value" "27nH"
 			(at 130.81 271.018 90)
 			(show_name no)
@@
 			)
 		)
-		(property "Value" "2.7nH"
+		(property "Value" "27nH"
 			(at 154.94 271.018 90)
 			(show_name no)
@@
 			)
 		)
-		(property "Value" "2.7nH"
+		(property "Value" "27nH"
 			(at 143.256 291.846 0)
 			(show_name no)
@@
 			)
 		)
-		(property "Value" "2.7nH"
+		(property "Value" "47nH"
 			(at 168.91 277.368 90)
 			(show_name no)

Commit message: fahh
Parts:
- added C106: 10uf, symbol Device:C
- added C107: 100nf, symbol Device:C
- added FB2: FerriteBead, symbol Device:FerriteBead
- L11: value 2.7nH -> 23nH
Connections:
- net GND: now also C106.2, C107.2, FB2.2; no longer P2.SH (SHIELD)
- net VDD33: now also C106.1, C107.1
- new net: FB2.1, P2.SH (SHIELD)
Other:
- moved on the sheet: D4

Commit message: adg
Parts:
- FB2: value FerriteBead -> BLM21PG221SN1D
Changed lines of the file:
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@@
 		(dnp no)
 		(property "Reference" "FB2"
-			(at 417.322 414.782 0)
+			(at 418.338 419.354 0)
 			(show_name no)
 			(do_not_autoplace no)
@@
 			)
 		)
-		(property "Value" "FerriteBead"
-			(at 411.48 417.83 0)
+		(property "Value" "BLM21PG221SN1D"
+			(at 411.988 421.64 0)
 			(show_name no)
 			(do_not_autoplace no)

Commit message: rhh4i
Parts:
- FB1: value FerriteBead -> BLM21PG221SN1D
- FB2: footprint (none) -> Inductor_SMD:L_0603_1608Metric_Pad1.05x0.95mm_HandSolder
Changed lines of the file:
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@@
 			)
 		)
-		(property "Value" "FerriteBead"
+		(property "Value" "BLM21PG221SN1D"
 			(at 630.936 287.528 0)
 			(show_name no)
@@
 			)
 		)
-		(property "Footprint" ""
+		(property "Footprint" "Inductor_SMD:L_0603_1608Metric_Pad1.05x0.95mm_HandSolder"
 			(at 422.402 416.56 90)
 			(hide yes)
