File: flipper black PCB/Flipper black ki cad/.history/Flipper black ki cad.kicad_pcb (KiCad board)
At the start: 2 copper layers, 108.5 x 102 mm, 250 parts, among them J2 Value: DISP_3.5_WAVESHARE, P1 JST-2pin, P2 USB_C_Plug_USB2.0, Q1 MMBT2222A, Q2 FS8205A, SW1 boot, SW2 REST, SW3 BTN_POWER, SW4 BTN_OK, SW5 BTN_UP, SW6 BTN_DOWN, SW7 BTN_LEFT, SW8 BTN_RIGHT, U1 ESP32-S3, U10 BGA725L6, U11 TLV70018_SOT23-5, U12 TXB0102DCU, U13 MCP23017x-x-SS, U14 TSOP382xx, U15 TP4056, U16 PESD5V0L4UG,115, U17 AP2112K-3.3, U18 DW01A, U2 W25Q128JVS, U3 CC1101, U4 SX1276, U5 PE4259, U6 PE4259, U7 PN5321A3HN, U8 MAX-M8Q, U9 MASW-007221, X1 433MHz SAW Filter, X2 B3715 868MHz SAW Filter, Y1 40MHz SMD 3225, Y2 26 MHz SMD, Y3 32 MHz SMD, Y4 27.120 MHz

Commit message: yooo
Parts:
- removed C29, C30, C31, C32, C33, C34, C57: 100nf, Capacitor_SMD:C_0603_1608Metric_Pad1.08x0.95mm_HandSolder
- removed C35, C36: 15pf, Capacitor_SMD:C_0603_1608Metric_Pad1.08x0.95mm_HandSolder
- removed C37, C38, C39, C40, C41, C42, C43, C44, C45, C46: 3.3pf, Capacitor_SMD:C_0603_1608Metric_Pad1.08x0.95mm_HandSolder
- removed C47, C48, C61, C62: 1nf, Capacitor_SMD:C_0603_1608Metric_Pad1.08x0.95mm_HandSolder
- removed C49, C50, C51, C58: 2.2pf, Capacitor_SMD:C_0603_1608Metric_Pad1.08x0.95mm_HandSolder
- removed C52, C54, C64, C65: 1.8pf, Capacitor_SMD:C_0603_1608Metric_Pad1.08x0.95mm_HandSolder
- removed C53, C55, C56, C60: 1.5pf, Capacitor_SMD:C_0603_1608Metric_Pad1.08x0.95mm_HandSolder
- removed C59: 1.0pf, Capacitor_SMD:C_0603_1608Metric_Pad1.08x0.95mm_HandSolder
- removed C63: 1.5 pf, Capacitor_SMD:C_0603_1608Metric_Pad1.08x0.95mm_HandSolder
- removed C66: 1uF, Capacitor_SMD:C_0603_1608Metric_Pad1.08x0.95mm_HandSolder
- removed L12: 24nH, Inductor_SMD:L_0603_1608Metric_Pad1.05x0.95mm_HandSolder
- removed L13, L14, L24: 100nH, Inductor_SMD:L_0603_1608Metric_Pad1.05x0.95mm_HandSolder
- removed L15, L16, L17, L20: 120nH, Inductor_SMD:L_0603_1608Metric_Pad1.05x0.95mm_HandSolder
- removed L18, L19: 68nH, Inductor_SMD:L_0603_1608Metric_Pad1.05x0.95mm_HandSolder
- removed L21, L22, L23: 22nH, Inductor_SMD:L_0603_1608Metric_Pad1.05x0.95mm_HandSolder
- removed R10, R11, R12, R13, R14, R16, R8, R9: 0R, Resistor_SMD:R_0402_1005Metric
- removed R15: 1k, Resistor_SMD:R_0402_1005Metric
- removed R17: 10k, Resistor_SMD:R_0402_1005Metric
- removed SX1276, SX1276_1: 50ohm, Connector_Coaxial:U.FL_Hirose_U.FL-R-SMT-1_Vertical
- removed U4: SX1276, Package_DFN_QFN:QFN-28-1EP_6x6mm_P0.65mm_EP4.8x4.8mm
- removed U5, U6: PE4259, PE4259:SOT65P215X110-6N
- removed X1: 433MHz SAW Filter, SF2136E:RFM-SAW-3X3MM
- removed X2: B3715 868MHz SAW Filter, Filter:Filter_SAW_Epcos_DCC6C_3x3mm
- removed Y3: 32 MHz SMD, Crystal:Crystal_SMD_2016-4Pin_2.0x1.6mm
- added C108: 1uf, Capacitor_SMD:C_0603_1608Metric_Pad1.08x0.95mm_HandSolder, F.Cu at (335.7, 123.2)
- added C109: 100nf, Capacitor_SMD:C_0603_1608Metric_Pad1.08x0.95mm_HandSolder, F.Cu at (338.8, 123.2)
- added C110: 470nf, Capacitor_SMD:C_0603_1608Metric_Pad1.08x0.95mm_HandSolder, F.Cu at (332.7, 127.0)
- added C111: 10pf, Capacitor_SMD:C_0603_1608Metric_Pad1.08x0.95mm_HandSolder, F.Cu at (335.7, 127.0)
- added C112: 10pf, Capacitor_SMD:C_0603_1608Metric_Pad1.08x0.95mm_HandSolder, F.Cu at (338.7, 127.0)
- added C113: 100nf, Capacitor_SMD:C_0603_1608Metric_Pad1.08x0.95mm_HandSolder, F.Cu at (332.7, 135.2)
- added C114: 6.8pf, Capacitor_SMD:C_0603_1608Metric_Pad1.08x0.95mm_HandSolder, F.Cu at (329.7, 123.2)
- added C115: 8.2pf, Capacitor_SMD:C_0603_1608Metric_Pad1.08x0.95mm_HandSolder, F.Cu at (332.7, 123.2)
- added C116: 1nf, Capacitor_SMD:C_0603_1608Metric_Pad1.08x0.95mm_HandSolder, F.Cu at (329.2, 106.7)
- added C117: 5.6pf, Capacitor_SMD:C_0603_1608Metric_Pad1.08x0.95mm_HandSolder, F.Cu at (332.7, 131.0)
- added C118: 10pf, Capacitor_SMD:C_0603_1608Metric_Pad1.08x0.95mm_HandSolder, F.Cu at (335.7, 131.0)
- added C119: 22pf, Capacitor_SMD:C_0603_1608Metric_Pad1.08x0.95mm_HandSolder, F.Cu at (338.7, 131.3)
- added C120: 10pf, Capacitor_SMD:C_0603_1608Metric_Pad1.08x0.95mm_HandSolder, F.Cu at (335.7, 135.0)
- added C121: 100nf, Capacitor_SMD:C_0603_1608Metric_Pad1.08x0.95mm_HandSolder, F.Cu at (338.7, 135.0)
- added C122: 1nf, Capacitor_SMD:C_0603_1608Metric_Pad1.08x0.95mm_HandSolder, F.Cu at (329.2, 110.4)
- added C123: 10pf, Capacitor_SMD:C_0603_1608Metric_Pad1.08x0.95mm_HandSolder, F.Cu at (325.7, 112.2)
- added C124: 5.6pf, Capacitor_SMD:C_0603_1608Metric_Pad1.08x0.95mm_HandSolder, F.Cu at (322.7, 111.9)
- added C125: 8.2pf, Capacitor_SMD:C_0603_1608Metric_Pad1.08x0.95mm_HandSolder, F.Cu at (332.2, 103.2)
- added L28: 18nH, Inductor_SMD:L_0603_1608Metric_Pad1.05x0.95mm_HandSolder, F.Cu at (335.2, 111.4)
- added L29: 15nH, Inductor_SMD:L_0603_1608Metric_Pad1.05x0.95mm_HandSolder, F.Cu at (338.2, 111.4)
- added L30: 15nH, Inductor_SMD:L_0603_1608Metric_Pad1.05x0.95mm_HandSolder, F.Cu at (341.2, 111.4)
- added L31: 22nH, Inductor_SMD:L_0603_1608Metric_Pad1.05x0.95mm_HandSolder, F.Cu at (335.2, 107.2)
- added L32: 27nH, Inductor_SMD:L_0603_1608Metric_Pad1.05x0.95mm_HandSolder, F.Cu at (338.2, 107.2)
- added L33: 18nH, Inductor_SMD:L_0603_1608Metric_Pad1.05x0.95mm_HandSolder, F.Cu at (341.2, 107.3)
- added L34: 22nH, Inductor_SMD:L_0603_1608Metric_Pad1.05x0.95mm_HandSolder, F.Cu at (332.2, 106.9)
- added R46: 10k, Resistor_SMD:R_0402_1005Metric, F.Cu at (332.2, 113.0)
- added R47: 100R, Resistor_SMD:R_0402_1005Metric, F.Cu at (332.2, 110.0)
- added R48: 100R, Resistor_SMD:R_0402_1005Metric, F.Cu at (329.7, 113.5)
- added SX1262: 50ohm, Connector_Coaxial:U.FL_Hirose_U.FL-R-SMT-1_Vertical, F.Cu at (424.8, 31.1)
- added U19: SX1262IMLTRT, SX1262IMLTRT:QFN50P400X400X100-25N, F.Cu at (340.7, 117.3)
- added U20: PE4259, PE4259:SOT65P215X110-6N, F.Cu at (325.2, 108.5)
- added Y5: 32 MHz SMD, Crystal:Crystal_SMD_2016-4Pin_2.0x1.6mm, F.Cu at (333.7, 117.3)
- J2: moved to B.Cu
- P2: footprint Connector_USB:USB_C_Receptacle_XKB_U262-16XN-4BVC11 -> Connector_USB:USB_C_Receptacle_GCT_USB4105-xx-A_16P_TopMnt_Horizontal
- R6: value 499Ohm -> 499R
- moved PN532_ANT1 397.5 mm to (372.1, 35.2)
- moved PCB_ANT1 381.9 mm to (414.0, 30.5), turned to -90 degrees
- moved R6 313.4 mm to (322.7, 130.1)
- moved R5 313.3 mm to (322.7, 127.6)
- moved R4 313.2 mm to (322.7, 125.1)
- moved R3 313.0 mm to (322.7, 122.6)
- moved R2 312.9 mm to (322.7, 120.1)
- moved R1 312.8 mm to (322.7, 117.6)
- moved R_EN1 309.6 mm to (324.9, 117.6)
- moved C17 308.9 mm to (325.5, 133.1)
- moved R_BOOT1 308.8 mm to (325.0, 120.1)
- moved C16 308.5 mm to (305.0, 138.1)
- moved R_G45 308.4 mm to (325.0, 122.6)
- moved R_G46 308.1 mm to (324.9, 125.1)
- moved C6 306.9 mm to (305.2, 132.1)
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- renumbered R_RSTPD1 to R_38, R_GPIO45 to R_G45, R_GPIO46 to R_G46
Connections:
- R1 pad 2: SPIQ -> SX1262_BUSY
- R2 pad 2: SPID -> SX1262_DIO2
- R6 pad 1: Net-(U1-U0TXD) -> TP_UART_TX
- TP9 pad 1: TP_UART_RX -> GPS_RXD
- U1 pad 38: CS_SX1276 -> CS_SX1262
- U1 pad 44: SX1276_DIO0 -> SX1262_DIO1
- U1 pad 45: SX1276_RESET -> SX1262_RESET
- U1 pad 49: Net-(U1-U0TXD) -> TP_UART_TX
Other:
- board size 108.5 x 102 mm -> 305 x 146.4 mm
- copper layers 2 -> 4

Commit message: zeeha
Parts:
- moved GPS_ANT1 282.5 mm to (166.1, 71.5)
- moved PCB_ANT1 238.2 mm to (179.4, 71.5)
- moved SX1262 210.5 mm to (218.2, 71.5)
- moved PN532_ANT1 183.1 mm to (193.3, 74.8)
- moved C67 124.6 mm to (164.8, 83.5)
- moved C69 124.6 mm to (160.3, 89.4)
- moved C73 124.6 mm to (170.3, 95.0)
- moved C74 124.6 mm to (173.1, 95.0)
- moved C75 124.6 mm to (169.6, 82.5)
- moved C77 124.6 mm to (177.2, 87.5)
- moved C78 124.6 mm to (175.9, 80.8)
- moved C79 124.6 mm to (177.3, 91.4)
- moved C80 124.6 mm to (179.7, 83.8)
- moved C82 124.6 mm to (167.6, 95.0)
- moved C83 124.6 mm to (165.1, 95.0)
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Other:
- board size 305 x 146.4 mm -> 92.3 x 143 mm

Commit message: krgtj
Parts:
- moved J2 0.62 mm to (198.0, 72.1)
- moved PN532_ANT1 0.62 mm to (193.4, 75.4)
Changed lines of the file:
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@@
 		)
 		(property "Value" "MCP23017x-x-SS"
-			(at 0 6.05 90)
+			(at -1.989269 7.357176 90)
 			(layer "F.Fab")
 			(effects
@@
 	(footprint "ESP_Antenna:ESPRESSIF_ESP32_MIFA_2.4GHz_Right"
 		(layer "F.Cu")
-		(at 193.342824 74.760731)
+		(at 193.45 75.375)
 		(descr "https://www.espressif.com/sites/default/files/documentation/esp32_datasheet_en.pdf")
 		(tags "PCB antenna")
@@
 	(footprint "Connector_FFC-FPC:Amphenol_F32Q-1A7x1-11015_1x15-1MP_P0.5mm_Horizontal"
 		(layer "B.Cu")
-		(at 197.892824 71.510731)
+		(at 198 72.125)
 		(descr "Amphenol F32Q/T FPC connector, 15 top-side contacts, 0.5mm pitch, SMT, https://cdn.amphenol-icc.com/media/wysiwyg/files/drawing/f32q-f32t.pdf")
 		(tags "F32T")
@@
 		)
 		(property "Value" "Value: DISP_3.5_WAVESHARE"
-			(at -0.5 5.5 180)
+			(at -0.392824 4.739269 180)
 			(layer "B.Fab")
 			(effects

Commit message: yaya
Parts:
- moved IR_LEDs1 2.01 mm to (182.5, 140.0)
- moved IR_LEDs2 2.01 mm to (189.3, 140.0)
- moved IR_LEDs3 2.01 mm to (196.1, 140.0)
- moved PN532_ANT1 0.13 mm to (193.4, 75.5)
Routing:
- net GND: track 0.00 -> 109.6 mm, vias 0 -> 127
- added copper zone on In1.Cu, net GND

Commit message: fie
Parts:
- PN532_ANT1: footprint ESP_Antenna:ESPRESSIF_ESP32_MIFA_2.4GHz_Right -> NFC_ANTENNA:NFC_ANT; moved to B.Cu
- moved PN532_ANT1 61.3 mm to (168.5, 131.5), turned to -90 degrees
- moved J2 0.15 mm to (198.0, 72.0)
Routing:
- net VDD33: track 0.00 -> 52.7 mm, vias 0 -> 71
- net GND: track 109.6 -> 110.2 mm
- added copper zone on In2.Cu, net VDD33

Commit message: yaya
Parts:
- moved PN532_ANT1 23.0 mm to (146.0, 136.2)
Changed lines of the file:
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@@
 	(footprint "NFC_ANTENNA:NFC_ANT"
 		(layer "B.Cu")
-		(at 168.5 131.5 -90)
+		(at 146 136.25 -90)
 		(property "Reference" "PN532_ANT1"
-			(at -5.25 0.25 90)
+			(at 4 -3.75 90)
 			(layer "B.SilkS")
 			(effects
@@
 		)
 		(property "Value" "50ohm"
-			(at 0 0 90)
+			(at 6.25 0.75 90)
 			(layer "B.SilkS")
 			(effects

Commit message: yay
Parts:
- removed PN532_ANT1: 50ohm, NFC_ANTENNA:NFC_ANT
- added AE1: Antenna_Loop, KiCad_Package coil:NFC_45x45_N4_NXP_PN5180, B.Cu at (198.4, 106.8)
Connections:
- C78 pad 2: GND -> Net-(AE1-Pad1)
- C79 pad 2: GND -> Net-(AE1-Pad1)
- C80 pad 2: GND -> Net-(AE1-Pad2)
- C81 pad 1: GND -> Net-(AE1-Pad2)
Routing:
- net Net-(AE1-Pad2): track 0.00 -> 13.3 mm, vias 0 -> 3
- net Net-(AE1-Pad1): track 0.00 -> 13.2 mm, vias 0 -> 3
- net GND: track 110.2 -> 106.6 mm, vias 127 -> 123

Commit message: u
Routing:
- net PN532_RESET: track 0.00 -> 61.9 mm
- net PN532_IRQ: track 0.00 -> 49.4 mm, vias 0 -> 2
- net GPS_EXTINT: track 0.00 -> 49.2 mm, vias 0 -> 2
- net CS_PN532: track 0.00 -> 45.7 mm, vias 0 -> 2
- net Net-(AE1-Pad1): track 13.2 -> 15.7 mm
