File: flipper black PCB/Flipper black ki cad/.history/Flipper black ki cad.kicad_pcb (KiCad board)
At the start: 4 copper layers, 92.3 x 143 mm, 213 parts, among them J2 Value: DISP_3.5_WAVESHARE, P1 JST-2pin, P2 USB_C_Plug_USB2.0, Q1 MMBT2222A, Q2 FS8205A, SW1 boot, SW2 REST, SW3 BTN_POWER, SW4 BTN_OK, SW5 BTN_UP, SW6 BTN_DOWN, SW7 BTN_LEFT, SW8 BTN_RIGHT, U1 ESP32-S3, U10 BGA725L6, U11 TLV70018_SOT23-5, U12 TXB0102DCU, U13 MCP23017x-x-SS, U14 TSOP382xx, U15 TP4056, U16 PESD5V0L4UG,115, U17 AP2112K-3.3, U18 DW01A, U19 SX1262IMLTRT, U2 W25Q128JVS, U20 PE4259, U3 CC1101, U7 PN5321A3HN, U8 MAX-M8Q, U9 MASW-007221, Y1 40MHz SMD 3225, Y2 26 MHz SMD, Y4 27.120 MHz, Y5 32 MHz SMD

Commit message: uyy
Routing:
- net CS_SX1262: track 0.00 -> 31.0 mm
Changed lines of the file:
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@@
+	)
+	(segment
+		(start 205.342824 106.460731)
+		(end 207.710731 106.460731)
+		(width 0.2)
+		(layer "F.Cu")
+		(net "CS_SX1262")
+	)
+	(segment
+		(start 234.779593 109)
+		(end 235.152824 109.373231)
+		(width 0.2)
+		(layer "F.Cu")
+		(net "CS_SX1262")
+	)
+	(segment
+		(start 215 107)
+		(end 217 109)
+		(width 0.2)
+		(layer "F.Cu")
+		(net "CS_SX1262")
+	)
+	(segment
+		(start 208.25 107)
+		(end 215 107)
+		(width 0.2)
+		(layer "F.Cu")
+		(net "CS_SX1262")
+	)
+	(segment
+		(start 217 109)
+		(end 234.779593 109)
+		(width 0.2)
+		(layer "F.Cu")
+		(net "CS_SX1262")
+	)
+	(segment
+		(start 207.710731 106.460731)
+		(end 208.25 107)
+		(width 0.2)
+		(layer "F.Cu")
+		(net "CS_SX1262")
 	)
 	(segment

Commit message: kdhe
Parts:
- moved R5 1.23 mm to (209.6, 112.0)
- moved R4 0.23 mm to (209.6, 108.5)
Routing:
- net SPI_SCK: track 0.00 -> 129.2 mm, vias 0 -> 6
- net SPI_MISO: track 0.00 -> 126.4 mm, vias 0 -> 9
- net SPI_MOSI: track 0.00 -> 123.1 mm, vias 0 -> 11
- net USB_DN: track 0.00 -> 87.4 mm, vias 0 -> 2
- net USB_DP: track 0.00 -> 86.0 mm, vias 0 -> 2
- net DISP_MISO: track 0.00 -> 54.2 mm, vias 0 -> 3
- net GPS_TIMEPULSE: track 0.00 -> 46.2 mm, vias 0 -> 2
- net I2C_SCL: track 0.00 -> 40.8 mm, vias 0 -> 3
- net BTN_POWER: track 0.00 -> 30.2 mm
- net Net-(U1-SPIQ): track 0.00 -> 14.2 mm, vias 0 -> 2
- net Net-(U1-SPICLK): track 0.00 -> 12.7 mm, vias 0 -> 2
- net Net-(U1-SPID): track 0.00 -> 8.59 mm, vias 0 -> 2
- net Net-(Q2-~-Pad1): track 0.00 -> 5.76 mm
- net Net-(U1-SPIHD): track 0.00 -> 4.69 mm
- net Net-(U1-SPIWP): track 0.00 -> 4.33 mm, vias 0 -> 2
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
Commit message: yayay
Routing:
- net BTN_DOWN: track 0.00 -> 68.8 mm, vias 0 -> 2
- net FLASH_CLK: track 0.00 -> 22.5 mm, vias 0 -> 2
- net FLASH_IO2: track 0.00 -> 16.4 mm, vias 0 -> 4
- net FLASH_IO1: track 0.00 -> 15.5 mm, vias 0 -> 2
- net FLASH_IO0: track 0.00 -> 5.64 mm, vias 0 -> 3
- net VDD33: track 52.6 -> 56.5 mm, vias 71 -> 70
- net GPS_TIMEPULSE: track 46.2 -> 47.1 mm
- net SPI_MISO: track 126.4 -> 126.9 mm

Commit message: fajhh
Parts:
- moved AE1 0.45 mm to (198.0, 106.8)
Routing:
- net EN_BTN: track 0.00 -> 145.9 mm, vias 0 -> 10
- net BOOT_BTN: track 0.00 -> 130.7 mm, vias 0 -> 10
- net BTN_OK: track 0.00 -> 72.8 mm, vias 0 -> 6
- net BTN_UP: track 0.00 -> 69.0 mm, vias 0 -> 4
- net CS_CC1101: track 0.00 -> 65.0 mm, vias 0 -> 2
- net CC1101_GDO0: track 0.00 -> 61.3 mm, vias 0 -> 4
- net CC1101_GDO2: track 0.00 -> 49.8 mm, vias 0 -> 2
- net GPS_RESET: track 0.00 -> 41.2 mm, vias 0 -> 2
- net GPS_SCL: track 0.00 -> 38.1 mm, vias 0 -> 2
- net GPS_SDA: track 0.00 -> 35.6 mm, vias 0 -> 4
- net FLASH_IO3: track 0.00 -> 35.5 mm, vias 0 -> 4
- net FLASH_IO0: track 5.64 -> 28.4 mm, vias 3 -> 6
- net FLASH_CS: track 0.00 -> 14.6 mm, vias 0 -> 4
- net Net-(AE1-Pad2): track 13.3 -> 16.3 mm, vias 3 -> 4
- net SPI_MOSI: track 122.8 -> 125.8 mm
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
Commit message: rt
Parts:
- AE1: value Antenna_Loop -> PN532 ANT
- L25, L26: value 560nH -> 220nH
- moved C25 106.5 mm to (151.4, 141.2)
- moved C26 106.5 mm to (144.4, 147.2)
- moved C28 106.5 mm to (133.4, 146.8)
- moved C18 106.5 mm to (139.2, 143.8)
- moved C20 106.5 mm to (129.8, 137.6)
- moved C21 106.5 mm to (135.8, 143.8)
- moved C22 106.5 mm to (147.8, 144.8)
- moved C23 106.5 mm to (137.1, 146.8)
- moved C24 106.5 mm to (144.1, 144.8)
- moved C27 106.5 mm to (141.2, 145.1)
- moved L10 106.5 mm to (151.2, 137.6)
- moved L11 106.5 mm to (142.8, 141.6)
- moved L5 106.5 mm to (142.8, 137.6)
- moved L6 106.5 mm to (145.8, 137.6)
- moved L7 106.5 mm to (148.8, 137.6)
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Routing:
- net EN_BTN: track 145.9 -> 0.00 mm, vias 10 -> 0
- net BOOT_BTN: track 130.7 -> 0.00 mm, vias 10 -> 0
- net SPI_SCK: track 129.9 -> 0.00 mm, vias 6 -> 0
- net SPI_MISO: track 129.3 -> 0.00 mm, vias 9 -> 0
- net SPI_MOSI: track 125.8 -> 0.00 mm, vias 11 -> 0
- net GND: track 106.6 -> 0.00 mm, vias 123 -> 0
- net USB_DN: track 89.3 -> 0.00 mm, vias 2 -> 0
- net USB_DP: track 87.4 -> 0.00 mm, vias 2 -> 0
- net BTN_OK: track 72.8 -> 0.00 mm, vias 6 -> 0
- net BTN_UP: track 69.0 -> 0.00 mm, vias 4 -> 0
- net BTN_DOWN: track 68.8 -> 0.00 mm, vias 2 -> 0
- net CS_CC1101: track 65.0 -> 0.00 mm, vias 2 -> 0
- net PN532_RESET: track 64.5 -> 0.00 mm
- net CC1101_GDO0: track 61.3 -> 0.00 mm, vias 4 -> 0
- net VDD33: track 56.6 -> 0.00 mm, vias 70 -> 0
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
Commit message: ufhy
Parts:
- moved AE1 25.7 mm to (103.3, 132.0)
- moved C100 5.02 mm to (163.8, 103.5)
- moved C105 5.02 mm to (167.5, 106.4)
- moved C84 5.02 mm to (158.2, 113.2)
- moved C89 5.02 mm to (173.6, 101.8)
- moved C91 5.02 mm to (170.2, 104.6)
- moved C92 5.02 mm to (176.3, 108.4)
- moved C94 5.02 mm to (173.5, 112.4)
- moved C96 5.02 mm to (158.2, 117.0)
- moved C97 5.02 mm to (158.2, 123.5)
- moved FB1 5.02 mm to (170.2, 101.1)
- moved JP1 5.02 mm to (167.0, 103.5)
- moved L27 5.02 mm to (164.0, 106.4)
- moved R25 5.02 mm to (171.8, 98.9)
- moved R27 5.02 mm to (159.5, 110.1)
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
Commit message: yay
Parts:
- moved AE1 39.7 mm to (127.5, 100.5)
- moved R25 12.0 mm to (161.2, 104.8), turned to 0 degrees
- moved FL1 7.81 mm to (166.9, 104.0), turned to 180 degrees
- moved R24 6.56 mm to (170.2, 107.0)
- moved C91 6.25 mm to (164.0, 104.5), turned to 0 degrees
- moved C92 5.82 mm to (172.5, 104.0), turned to 180 degrees
- moved JP1 5.60 mm to (161.8, 101.3), turned to 0 degrees
- moved C100 5.11 mm to (159.0, 101.6)
- moved C89 5.11 mm to (168.5, 101.0)
- moved FB1 4.50 mm to (165.8, 101.1)
- moved U10 4.23 mm to (169.2, 104.0), turned to -90 degrees
- moved U9 4.22 mm to (171.8, 101.3)
- moved C94 3.74 mm to (177.1, 113.2), turned to 0 degrees
- moved C95 3.25 mm to (173.8, 130.2), turned to 0 degrees
- moved C98 2.83 mm to (159.0, 105.4)
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Routing:
- removed copper zone on In1.Cu, net GND
- removed copper zone on In2.Cu, net VDD33
Other:
- board size 92.3 x 143 mm -> 142.1 x 143 mm

Commit message: uu
Parts:
- moved R_38 139.6 mm to (119.3, 89.4)
- moved R18 135.1 mm to (123.3, 87.6)
- moved R19 134.7 mm to (123.3, 90.9)
- moved R21 133.9 mm to (115.5, 114.6)
- moved C69 133.5 mm to (116.0, 100.9)
- moved C75 133.0 mm to (127.7, 88.4), turned to 180 degrees
- moved R20 132.6 mm to (119.3, 97.4)
- moved R22 132.0 mm to (119.3, 102.6)
- moved L25 131.7 mm to (131.4, 88.4)
- moved C78 131.6 mm to (134.9, 88.4)
- moved C80 131.6 mm to (138.7, 91.4)
- moved C76 131.6 mm to (135.1, 91.4)
- moved C81 131.6 mm to (138.6, 88.4)
- moved L26 131.6 mm to (131.7, 91.4)
- moved R_I0 131.5 mm to (118.5, 114.6)
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Routing:
- added copper zone on In1.Cu, net GND
- added copper zone on In2.Cu, net VDD33
