File: flipper black PCB/Flipper black ki cad/.history/Flipper black ki cad.kicad_pcb (KiCad board)
At the start: 4 copper layers, 142.1 x 143 mm, 213 parts, among them J2 Value: DISP_3.5_WAVESHARE, P1 JST-2pin, P2 USB_C_Plug_USB2.0, Q1 MMBT2222A, Q2 FS8205A, SW1 boot, SW2 REST, SW3 BTN_POWER, SW4 BTN_OK, SW5 BTN_UP, SW6 BTN_DOWN, SW7 BTN_LEFT, SW8 BTN_RIGHT, U1 ESP32-S3, U10 BGA725L6, U11 TLV70018_SOT23-5, U12 TXB0102DCU, U13 MCP23017x-x-SS, U14 TSOP382xx, U15 TP4056, U16 PESD5V0L4UG,115, U17 AP2112K-3.3, U18 DW01A, U19 SX1262IMLTRT, U2 W25Q128JVS, U20 PE4259, U3 CC1101, U7 PN5321A3HN, U8 MAX-M8Q, U9 MASW-007221, Y1 40MHz SMD 3225, Y2 26 MHz SMD, Y4 27.120 MHz, Y5 32 MHz SMD

Commit message: yayay
Parts:
- moved C78 42.5 mm to (177.2, 84.7)
- moved C68 38.5 mm to (175.5, 100.7), turned to 180 degrees
- moved C69 38.5 mm to (154.3, 97.1)
- moved C70 38.5 mm to (157.8, 106.4), turned to 180 degrees
- moved C71 38.5 mm to (175.5, 95.1), turned to 180 degrees
- moved C72 38.5 mm to (175.5, 97.7)
- moved C74 38.5 mm to (172.3, 106.9), turned to -90 degrees
- moved C77 38.5 mm to (178.2, 96.2), turned to 90 degrees
- moved C79 38.5 mm to (178.3, 100.0)
- moved C82 38.5 mm to (165.9, 106.9), turned to 90 degrees
- moved R18 38.5 mm to (161.6, 83.9)
- moved R20 38.5 mm to (157.6, 93.7)
- moved R_38 38.5 mm to (157.6, 85.7)
- moved Y4 38.5 mm to (177.9, 103.8)
- moved C75 38.5 mm to (166.1, 84.7), turned to 0 degrees
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
Commit message: hyydge
Parts:
- moved C102 0.72 mm to (220.2, 202.7)
- moved C101 0.25 mm to (216.4, 202.7)
Routing:
- net GND: track 0.00 -> 219.9 mm, vias 0 -> 74
- net VDD33: track 0.00 -> 0.92 mm, vias 0 -> 1

Commit message: sivk
Parts:
- moved C_EN1 2.28 mm to (192.3, 94.0)
- moved L2 2.14 mm to (199.9, 96.4)
- moved L4 2.11 mm to (196.3, 96.4), turned to 180 degrees
- moved L1 1.70 mm to (199.9, 94.6)
- moved L3 1.67 mm to (196.3, 94.6)
- moved C17 1.16 mm to (213.8, 109.3)
- moved R5 1.16 mm to (211.5, 109.3)
- moved R6 1.16 mm to (211.5, 110.6)
- moved R4 0.80 mm to (209.9, 103.8)
- moved R_G46 0.80 mm to (212.3, 103.8)
- moved R1 0.68 mm to (210.0, 96.6)
- moved R_EN1 0.68 mm to (212.2, 96.6)
- moved R2 0.66 mm to (210.0, 99.1)
- moved R3 0.66 mm to (210.0, 101.6)
- moved R_BOOT1 0.66 mm to (212.2, 99.1)
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Routing:
- net EN_BTN: track 0.00 -> 152.8 mm, vias 0 -> 4
- net GPS_RXD: track 0.00 -> 139.7 mm, vias 0 -> 6
- net BOOT_BTN: track 0.00 -> 127.3 mm, vias 0 -> 4
- net SPI_MISO: track 0.00 -> 117.5 mm, vias 0 -> 10
- net USB_DN: track 0.00 -> 116.2 mm, vias 0 -> 6
- net USB_DP: track 0.00 -> 113.9 mm, vias 0 -> 6
- net TP_UART_TX: track 0.00 -> 101.5 mm, vias 0 -> 5
- net VDD33: track 0.92 -> 98.3 mm, vias 1 -> 54
- net SPI_SCK: track 0.00 -> 78.3 mm, vias 0 -> 7
- net BTN_OK: track 0.00 -> 73.9 mm
- net PN532_RESET: track 0.00 -> 66.8 mm, vias 0 -> 3
- net BTN_UP: track 0.00 -> 63.9 mm
- net BTN_RIGHT: track 0.00 -> 60.7 mm, vias 0 -> 2
- net GPS_TIMEPULSE: track 0.00 -> 59.1 mm, vias 0 -> 4
- net Net-(U1-LNA_IN): track 0.00 -> 58.5 mm, vias 0 -> 7
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
Commit message: zeeeee
yayaya
Parts:
- moved C15 24.4 mm to (183.6, 96.8)
- moved C17 10.6 mm to (216.0, 119.7)
- moved Y4 0.96 mm to (177.2, 103.2)
- moved C18 0.51 mm to (228.3, 83.7)
- moved R46 0.40 mm to (168.2, 126.9)
- moved R47 0.40 mm to (168.2, 124.7)
- turned AE1 to -90 degrees
Routing:
- net IR_TX: track 0.00 -> 154.0 mm, vias 0 -> 9
- net +5V: track 0.00 -> 143.6 mm
- net SPI_MOSI: track 0.00 -> 134.3 mm, vias 0 -> 10
- net TP_BAT: track 0.00 -> 120.9 mm, vias 0 -> 7
- net SX1262_DIO2: track 0.00 -> 101.7 mm, vias 0 -> 11
- net BTN_DOWN: track 0.00 -> 101.0 mm, vias 0 -> 8
- net FLASH_CLK: track 0.00 -> 91.2 mm, vias 0 -> 12
- net SX1262_BUSY: track 0.00 -> 89.5 mm, vias 0 -> 8
- net Net-(SX1262-A): track 0.00 -> 89.5 mm
- net FLASH_IO1: track 0.00 -> 85.5 mm, vias 0 -> 12
- net FLASH_IO2: track 0.00 -> 82.0 mm, vias 0 -> 12
- net Net-(U20-RF1): track 0.00 -> 68.7 mm, vias 0 -> 4
- net +1V8: track 0.00 -> 66.3 mm, vias 0 -> 4
- net Net-(Y1-XIN): track 0.00 -> 60.4 mm, vias 0 -> 4
- net Net-(C117-Pad2): track 0.00 -> 56.4 mm, vias 0 -> 2
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