File: flipper black PCB/Flipper black ki cad/Flipper black ki cad.kicad_sch (KiCad schematic)
At the start: 246 parts, among them J1 Barrel_Jack, J2 Value: DISP_3.5_WAVESHARE, P1 JST-2pin, P2 USB_C_Plug_USB2.0, Q1 MMBT2222A, Q2 FS8205A, SW1 SW_Push, SW2 SW_Push, SW3 BTN_POWER, SW4 BTN_OK, SW5 BTN_UP, SW6 BTN_DOWN, SW7 BTN_LEFT, SW8 BTN_RIGHT, U1 ESP32-S3, U10 BGA725L6, U11 TLV70018_SOT23-5, U12 TXB0102DCU, U13 MCP23017x-x-SS, U14 TSOP382xx, U15 TP4056, U17 AP2112K-3.3, U18 DW01A, U2 W25Q128JVS, U3 CC1101, U4 SX1276, U5 PE4259, U6 PE4259, U7 PN5321A3HN, U8 MAX-M8Q, U9 MASW-007221, X1 B3715 868MHz SAW Filter, X2 B3715 868MHz SAW Filter, Y1 40MHz SMD 3225, Y2 26 MHz SMD, Y3 32 MHz SMD, Y4 27.120 MHz

Commit message: fahhh
Parts:
- removed TP6: TestPoint, symbol Connector:TestPoint
- TP1: value TestPoint -> TP_3V3
- TP10: value TestPoint -> TP_RESET
- TP2: value TestPoint -> TP_BAT
- TP3: value TestPoint -> TP_5V
- TP4: value TestPoint -> TP_GND
- TP5: value TestPoint -> TP_BOOT
- TP7: value TestPoint -> TP_IR_TX
Connections:
- net +3V3: now also TP1.1
- net +5V: now also TP3.1
- net BOOT_BTN: now also TP5.1
- net EN_BTN: now also TP10.1
- net GND: now also TP4.1
- net IR_TX: now also TP7.1
- net TP_BAT: now reaches C101.1, P1.1, U15.5 (BAT), U18.5 (VCC)
- net TP_BAT: now also TP2.1
Other:
- moved on the sheet: R34

Commit message: fah
Parts:
- TP8: value TestPoint -> TP_UART_TX
- TP9: value TestPoint -> TP_UART_RX
Connections:
- net TP_UART_TX: now reaches R6.1, U1.49 (U0TXD)
- net TP_UART_TX: now also TP8.1
- net TP_UART_RX: now reaches TP9.1
Other:
- moved on the sheet: R6
Changed lines of the file:
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@@
 	(wire
 		(pts
+			(xy 736.6 408.94) (xy 736.6 415.29)
+		)
+		(stroke
+			(width 0)
+			(type default)
+		)
+	)
+	(wire
+		(pts
 			(xy 74.93 377.19) (xy 82.55 377.19)
 		)
@@
 	(wire
 		(pts
-			(xy 173.99 135.89) (xy 182.88 135.89)
+			(xy 175.26 135.89) (xy 182.88 135.89)
 		)
 		(stroke
@@
 	(wire
 		(pts
-			(xy 151.13 135.89) (xy 166.37 135.89)
+			(xy 151.13 135.89) (xy 167.64 135.89)
 		)
 		(stroke
@@
 	(wire
 		(pts
+			(xy 711.2 408.94) (xy 711.2 415.29)
+		)
+		(stroke
+			(width 0)
+			(type default)
+		)
+	)
+	(wire
+		(pts
 			(xy 204.47 416.56) (xy 204.47 419.1)
 		)
@@
 		)
 	)
+	(global_label "TP_UART_TX"
+		(shape input)
+		(at 151.13 135.89 0)
+		(fields_autoplaced yes)
+		(effects
+			(font
+				(size 1.27 1.27)
+				(thickness 0.1588)
+			)
+			(justify left)
+		)
+		(property "Intersheetrefs" "${INTERSHEET_REFS}"
+			(at 165.1218 135.89 0)
+			(hide yes)
+			(show_name no)
+			(do_not_autoplace no)
+			(effects
+				(font
+					(size 1.27 1.27)
+				)
+				(justify left)
+			)
+		)
+	)
 	(global_label "BTN_UP"
 		(shape input)
@@
 			(font
 				(size 1.27 1.27)
-				(thickness 0.254)
-				(bold yes)
+				(thickness 0.1588)
 			)
 			(justify left)
 		)
 		(property "Intersheetrefs" "${INTERSHEET_REFS}"
-			(at 771.9926 379.73 0)
+			(at 771.5166 379.73 0)
 			(hide yes)
 			(show_name no)
@@
 		)
 	)
+	(global_label "TP_UART_RX"
+		(shape input)
+		(at 711.2 415.29 0)
+		(fields_autoplaced yes)
+		(effects
+			(font
+				(size 1.27 1.27)
+				(thickness 0.1588)
+			)
+			(justify left)
+		)
+		(property "Intersheetrefs" "${INTERSHEET_REFS}"
+			(at 725.4942 415.29 0)
+			(hide yes)
+			(show_name no)
+			(do_not_autoplace no)
+			(effects
+				(font
+					(size 1.27 1.27)
+				)
+				(justify left)
+			)
+		)
+	)
 	(global_label "BTN_POWER"
 		(shape input)
@@
 		)
 	)
+	(global_label "TP_UART_TX"
+		(shape input)
+		(at 736.6 415.29 0)
+		(fields_autoplaced yes)
+		(effects
+			(font
+				(size 1.27 1.27)
+				(thickness 0.254)
+				(bold yes)
+			)
+			(justify left)
+		)
+		(property "Intersheetrefs" "${INTERSHEET_REFS}"
+			(at 751.0678 415.29 0)
+			(hide yes)
+			(show_name no)
+			(do_not_autoplace no)
+			(effects
+				(font
+					(size 1.27 1.27)
+				)
+				(justify left)
+			)
+		)
+	)
 	(global_label "RXTX RF sx"
 		(shape input)
@@
 	(symbol
 		(lib_id "Device:R_US")
-		(at 170.18 135.89 90)
+		(at 171.45 135.89 90)
 		(unit 1)
 		(body_style 1)
@@
 		(dnp no)
 		(property "Reference" "R6"
-			(at 165.608 134.874 90)
+			(at 167.894 135.128 90)
 			(show_name no)
 			(do_not_autoplace no)
@@
 		)
 		(property "Value" "499Ohm"
-			(at 176.276 134.62 90)
+			(at 177.8 134.874 90)
 			(show_name no)
 			(do_not_autoplace no)
@@
 		)
 		(property "Footprint" ""
-			(at 170.434 134.874 90)
+			(at 171.704 134.874 90)
 			(hide yes)
 			(show_name no)
@@
 		)
 		(property "Datasheet" ""
-			(at 170.18 135.89 0)
+			(at 171.45 135.89 0)
 			(hide yes)
 			(show_name no)
@@
 		)
 		(property "Description" "Resistor, US symbol"
-			(at 170.18 135.89 0)
+			(at 171.45 135.89 0)
 			(hide yes)
 			(show_name no)
@@
 			)
 		)
-		(property "Value" "TestPoint"
+		(property "Value" "TP_UART_RX"
 			(at 713.74 406.9079 0)
 			(show_name no)
@@
 			)
 		)
-		(property "Value" "TestPoint"
+		(property "Value" "TP_UART_TX"
 			(at 739.14 406.9079 0)
 			(show_name no)

Commit message: more more more
Connections:
- net TP_UART_RX is gone; now on net GPS_RXD: TP9.1
Changed lines of the file:
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@@
+		)
+	)
+	(global_label "TP_UART_RX"
+		(shape input)
+		(at 151.13 138.43 0)
+		(fields_autoplaced yes)
+		(effects
+			(font
+				(size 1.27 1.27)
+				(thickness 0.1588)
+			)
+			(justify left)
+		)
+		(property "Intersheetrefs" "${INTERSHEET_REFS}"
+			(at 165.4242 138.43 0)
+			(hide yes)
+			(show_name no)
+			(do_not_autoplace no)
+			(effects
+				(font
+					(size 1.27 1.27)
+				)
+				(justify left)
+			)
 		)
 	)
@@
 			(font
 				(size 1.27 1.27)
-				(thickness 0.254)
-				(bold yes)
-			)
-			(justify left)
-		)
-		(property "Intersheetrefs" "${INTERSHEET_REFS}"
-			(at 751.0678 415.29 0)
-			(hide yes)
-			(show_name no)
+				(thickness 0.1588)
+			)
+			(justify left)
+		)
+		(property "Intersheetrefs" "${INTERSHEET_REFS}"
+			(at 750.5918 415.29 0)
+			(hide yes)
+			(show_name no)
