File: flipper black PCB/Flipper black ki cad/Flipper black ki cad.kicad_sch (KiCad schematic)
At the start: 246 parts, among them J1 Barrel_Jack, J2 Value: DISP_3.5_WAVESHARE, P1 JST-2pin, P2 USB_C_Plug_USB2.0, Q1 MMBT2222A, Q2 FS8205A, SW1 SW_Push, SW2 SW_Push, SW3 BTN_POWER, SW4 BTN_OK, SW5 BTN_UP, SW6 BTN_DOWN, SW7 BTN_LEFT, SW8 BTN_RIGHT, U1 ESP32-S3, U10 BGA725L6, U11 TLV70018_SOT23-5, U12 TXB0102DCU, U13 MCP23017x-x-SS, U14 TSOP382xx, U15 TP4056, U16 PESD5V0L4UG,115, U17 AP2112K-3.3, U18 DW01A, U2 W25Q128JVS, U3 CC1101, U4 SX1276, U5 PE4259, U6 PE4259, U7 PN5321A3HN, U8 MAX-M8Q, U9 MASW-007221, X1 B3715 868MHz SAW Filter, X2 B3715 868MHz SAW Filter, Y1 40MHz SMD 3225, Y2 26 MHz SMD, Y3 32 MHz SMD, Y4 27.120 MHz

Commit message: sui
Parts:
- C1, C10, C100, C101, C104, C11, C12, C13, C15, C16, C17, C18, C19, C2, C20, C21, C22, C23, C24, C28, C29, C3, C30, C31, C32, C33, C34, C35, C36, C37, C38, C39, C4, C40, C41, C42, C43, C44, C45, C46, C47, C48, C49, C5, C50, C51, C52, C53, C54, C55, C56, C57, C58, C59, C6, C60, C61, C62, C63, C64, C65, C66, C67, C68, C69, C7, C70, C71, C72, C73, C74, C75, C76, C77, C78, C79, C8, C80, C81, C82, C83, C84, C85, C86, C87, C88, C89, C9, C90, C93, C94, C95, C96, C97, C98, C99, C_EN1: footprint (none) -> Capacitor_SMD:C_0603_1608Metric_Pad1.08x0.95mm_HandSolder
- C102, C103: value C -> 10uf; footprint (none) -> Capacitor_SMD:C_0603_1608Metric_Pad1.08x0.95mm_HandSolder
- C14, C25: value 1.0 pF -> 1.0pF; footprint (none) -> Capacitor_SMD:C_0603_1608Metric_Pad1.08x0.95mm_HandSolder
- C26: value 1.5 pf -> 1.5pf; footprint (none) -> Capacitor_SMD:C_0603_1608Metric_Pad1.08x0.95mm_HandSolder
- C27: value 1.5 pF -> 1.5pF; footprint (none) -> Capacitor_SMD:C_0603_1608Metric_Pad1.08x0.95mm_HandSolder
- C91: value C -> 1nf; footprint (none) -> Capacitor_SMD:C_0603_1608Metric_Pad1.08x0.95mm_HandSolder
- C92: value C -> 22pf; footprint (none) -> Capacitor_SMD:C_0603_1608Metric_Pad1.08x0.95mm_HandSolder
- R1, R10, R11, R12, R14, R15, R16, R17, R18, R19, R2, R20, R21, R22, R23, R24, R25, R27, R28, R29, R3, R30, R31, R32, R33, R34, R35, R36, R37, R38, R39, R4, R40, R41, R42, R43, R44, R5, R6, R7, R8, R9, R_BOOT1, R_EN1, R_GPIO45, R_GPIO46, R_I0, R_I1, R_RSTPD1: footprint (none) -> Resistor_SMD:R_0402_1005Metric
- R13: value NC -> 0R; footprint (none) -> Resistor_SMD:R_0402_1005Metric
- R26: value R -> 10K; footprint (none) -> Resistor_SMD:R_0402_1005Metric
- SW1: value SW_Push -> boot
- SW2: value SW_Push -> REST
- Y1, Y2, Y3, Y4: footprint (none) -> Crystal:Crystal_SMD_2016-4Pin_2.0x1.6mm

Commit message: sui
Parts:
- CC1101_ANT1, GPS_ANT1, PCB_ANT1, SX1276, SX1276_1: footprint (none) -> Connector_Coaxial:U.FL_Hirose_U.FL-R-SMT-1_Vertical
- D1: footprint (none) -> Diode_SMD:D_SOD-323_HandSoldering
- D2, D3: footprint (none) -> LED_SMD:LED_0603_1608Metric_Pad1.05x0.95mm_HandSolder
- FB1, L1, L10, L11, L12, L13, L14, L15, L16, L17, L18, L19, L2, L20, L21, L22, L23, L24, L25, L26, L27, L3, L4, L5, L6, L7, L8, L9: footprint (none) -> Inductor_SMD:L_0603_1608Metric_Pad1.05x0.95mm_HandSolder
- J1: footprint (none) -> Connector_BarrelJack:BarrelJack_Wuerth_694108106102_2.5x5.5mm
- J2: footprint (none) -> Connector_FFC-FPC:Amphenol_F32Q-1A7x1-11015_1x15-1MP_P0.5mm_Horizontal
- JP1: footprint (none) -> Jumper:SolderJumper-2_P1.3mm_Bridged2Bar_Pad1.0x1.5mm
- P1: footprint JST_PHR-2 -> Connector_JST:JST_EH_S3B-EH_1x03_P2.50mm_Horizontal
- P2: footprint (none) -> Connector_USB:USB_C_Receptacle_XKB_U262-16XN-4BVC11
- PN532_ANT1: footprint (none) -> ESP_Antenna:ESPRESSIF_ESP32_MIFA_2.4GHz_Right
- SW1, SW2: footprint (none) -> Button_Switch_SMD:SW_SPST_B3U-1000P
- SW3, SW4, SW5, SW6, SW7, SW8: footprint (none) -> Button_Switch_SMD:Nidec_Copal_SH-7010B
Other:
- moved on the sheet: C44, C45, L18

Commit message: no finally
Parts:
- SW3, SW4, SW5, SW6, SW7, SW8: footprint Button_Switch_SMD:Nidec_Copal_SH-7010B -> Button_Switch_SMD:SW_DIP_SPSTx01_Slide_6.7x4.1mm_W6.73mm_P2.54mm_LowProfile_JPin
- TP1, TP10, TP2, TP3, TP4, TP5, TP7, TP8, TP9: footprint (none) -> TestPoint:TestPoint_2Pads_Pitch2.54mm_Drill0.8mm
- U10: footprint (none) -> BGA725L6E6327:BGA725L6E6327
Changed lines of the file:
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@@
 			)
 		)
-		(property "Footprint" ""
+		(property "Footprint" "TestPoint:TestPoint_2Pads_Pitch2.54mm_Drill0.8mm"
 			(at 690.88 408.94 0)
 			(hide yes)
@@
 			)
 		)
-		(property "Footprint" ""
+		(property "Footprint" "TestPoint:TestPoint_2Pads_Pitch2.54mm_Drill0.8mm"
 			(at 741.68 375.92 0)
 			(hide yes)
@@
 			)
 		)
-		(property "Footprint" "Button_Switch_SMD:Nidec_Copal_SH-7010B"
+		(property "Footprint" "Button_Switch_SMD:SW_DIP_SPSTx01_Slide_6.7x4.1mm_W6.73mm_P2.54mm_LowProfile_JPin"
 			(at 588.01 396.24 0)
 			(hide yes)
@@
 			)
 		)
-		(property "Footprint" ""
+		(property "Footprint" "TestPoint:TestPoint_2Pads_Pitch2.54mm_Drill0.8mm"
 			(at 767.08 408.94 0)
 			(hide yes)
@@
 			)
 		)
-		(property "Footprint" "Button_Switch_SMD:Nidec_Copal_SH-7010B"
+		(property "Footprint" "Button_Switch_SMD:SW_DIP_SPSTx01_Slide_6.7x4.1mm_W6.73mm_P2.54mm_LowProfile_JPin"
 			(at 636.27 397.51 0)
 			(hide yes)
@@
 			)
 		)
-		(property "Footprint" "Button_Switch_SMD:Nidec_Copal_SH-7010B"
+		(property "Footprint" "Button_Switch_SMD:SW_DIP_SPSTx01_Slide_6.7x4.1mm_W6.73mm_P2.54mm_LowProfile_JPin"
 			(at 544.83 368.3 0)
 			(hide yes)
@@
 			)
 		)
-		(property "Footprint" "Button_Switch_SMD:Nidec_Copal_SH-7010B"
+		(property "Footprint" "Button_Switch_SMD:SW_DIP_SPSTx01_Slide_6.7x4.1mm_W6.73mm_P2.54mm_LowProfile_JPin"
 			(at 544.83 396.24 0)
 			(hide yes)
@@
 			)
 		)
-		(property "Footprint" "Button_Switch_SMD:Nidec_Copal_SH-7010B"
+		(property "Footprint" "Button_Switch_SMD:SW_DIP_SPSTx01_Slide_6.7x4.1mm_W6.73mm_P2.54mm_LowProfile_JPin"
 			(at 636.27 369.57 0)
 			(hide yes)
@@
 			)
 		)
-		(property "Footprint" ""
+		(property "Footprint" "TestPoint:TestPoint_2Pads_Pitch2.54mm_Drill0.8mm"
 			(at 716.28 408.94 0)
 			(hide yes)
@@
 			)
 		)
-		(property "Footprint" ""
+		(property "Footprint" "TestPoint:TestPoint_2Pads_Pitch2.54mm_Drill0.8mm"
 			(at 741.68 408.94 0)
 			(hide yes)
@@
 			)
 		)
-		(property "Footprint" ""
+		(property "Footprint" "TestPoint:TestPoint_2Pads_Pitch2.54mm_Drill0.8mm"
 			(at 690.88 375.92 0)
 			(hide yes)
@@
 			)
 		)
-		(property "Footprint" ""
+		(property "Footprint" "TestPoint:TestPoint_2Pads_Pitch2.54mm_Drill0.8mm"
 			(at 767.08 375.92 0)
 			(hide yes)
@@
 			)
 		)
-		(property "Footprint" ""
+		(property "Footprint" "TestPoint:TestPoint_2Pads_Pitch2.54mm_Drill0.8mm"
 			(at 716.28 375.92 0)
 			(hide yes)
@@
 			)
 		)
-		(property "Footprint" "Button_Switch_SMD:Nidec_Copal_SH-7010B"
+		(property "Footprint" "Button_Switch_SMD:SW_DIP_SPSTx01_Slide_6.7x4.1mm_W6.73mm_P2.54mm_LowProfile_JPin"
 			(at 588.01 368.3 0)
 			(hide yes)
@@
 			)
 		)
-		(property "Footprint" ""
+		(property "Footprint" "TestPoint:TestPoint_2Pads_Pitch2.54mm_Drill0.8mm"
 			(at 792.48 375.92 0)
 			(hide yes)
@@
 			)
 		)
-		(property "Footprint" ""
+		(property "Footprint" "BGA725L6E6327:BGA725L6E6327"
 			(at 681.99 309.88 0)
 			(hide yes)

Commit message: yoo
Connections:
- net +3.3V: no longer R27.1
- net +3V3: no longer C102.1, C103.1, C99.1, R26.1, R28.1, U12.7 (VCCB), U17.5 (VOUT)
- net VDD33: now also C102.1, C103.1, C99.1, R26.1, R27.1, R28.1, U12.7 (VCCB), U17.5 (VOUT); no longer C3.1, L1.2, U1.2 (VDD3P3), U1.3 (VDD3P3)
- new net: C3.1, L1.2, U1.2 (VDD3P3), U1.3 (VDD3P3)

Commit message: fahh
Parts:
- removed X1: B3715 868MHz SAW Filter, Filter:Filter_SAW_Epcos_DCC6C_3x3mm, symbol RF_Filter:B3715
- added FIL1: SF2136E, RFM-SAW-3X3MM, symbol SF2136E:SF2136E
- TP1: value TP_3V3 -> TP_VDD33
Connections:
- net +3.3V is gone; now on net VDD33: R_RSTPD1.1
- net +3V3 is gone; now on net VDD33: C94.1, C95.1, J2.1 (Pin_1), J2.2 (Pin_2), TP1.1, U11.1 (IN)
- net GND: now also FIL1.1 (GND), FIL1.3 (GND), FIL1.4 (GND), FIL1.6 (GND)
- net GPS_RXD: no longer U12.5 (A1), U8.3 (RXD)
- net GPS_TXD: no longer U12.4 (A2), U8.2 (TXD)
- net at R10.2, R8.2, R9.2: now also FIL1.5 (OUT)
- net at R11.1, R12.2, R13.2: now also FIL1.2 (IN)
- new net GPS_RX_1V8: U12.4 (A2), U8.3 (RXD)
- new net GPS_TX_1V8: U12.5 (A1), U8.2 (TXD)
Other:
- moved on the sheet: R10, R11

Commit message: yooohhohoh
Parts:
- removed J1: Barrel_Jack, Connector_BarrelJack:BarrelJack_Wuerth_694108106102_2.5x5.5mm, symbol Connector:Barrel_Jack
- added C105: 100pf, symbol Device:C
- X1: renamed from FIL1; value SF2136E -> 433MHz SAW Filter
Connections:
- net at FB1.2: now also C91.2
- net at L27.2: now also C105.1; no longer U10.5 (AI)
- new net: C105.2, U10.5 (AI)
Other:
- moved on the sheet: GPS_ANT1, L27
Changed lines of the file:
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@@
 	(wire
 		(pts
-			(xy 708.66 307.34) (xy 708.66 309.88)
+			(xy 712.47 294.64) (xy 712.47 297.18)
 		)
 		(stroke
@@
 	(wire
 		(pts
-			(xy 708.66 294.64) (xy 708.66 299.72)
+			(xy 712.47 281.94) (xy 712.47 287.02)
 		)
 		(stroke
@@
 		)
 	)
+	(wire
+		(pts
+			(xy 712.47 304.8) (xy 712.47 309.88)
+		)
+		(stroke
+			(width 0)
+			(type default)
+		)
+	)
 	(polyline
 		(pts
@@
 	(wire
 		(pts
-			(xy 628.65 300.99) (xy 613.41 300.99)
-		)
-		(stroke
-			(width 0)
-			(type default)
-		)
-	)
-	(wire
-		(pts
 			(xy 393.7 234.95) (xy 401.32 234.95)
 		)
@@
 	(wire
 		(pts
-			(xy 694.69 309.88) (xy 708.66 309.88)
+			(xy 694.69 309.88) (xy 712.47 309.88)
 		)
 		(stroke
@@
 	(wire
 		(pts
-			(xy 603.25 300.99) (xy 608.33 300.99)
+			(xy 603.25 300.99) (xy 628.65 300.99)
 		)
 		(stroke
@@
 	(symbol
 		(lib_id "Device:Antenna")
-		(at 708.66 289.56 0)
+		(at 712.47 276.86 0)
 		(unit 1)
 		(body_style 1)
@@
 		(in_pos_files yes)
 		(dnp no)
-		(fields_autoplaced yes)
 		(property "Reference" "GPS_ANT1"
-			(at 711.2 288.9249 0)
+			(at 708.914 270.256 0)
 			(show_name no)
 			(do_not_autoplace no)
@@
 		)
 		(property "Value" "50ohm"
-			(at 711.2 291.4649 0)
+			(at 708.914 272.796 0)
 			(show_name no)
 			(do_not_autoplace no)
@@
 		)
 		(property "Footprint" "Connector_Coaxial:U.FL_Hirose_U.FL-R-SMT-1_Vertical"
-			(at 708.66 289.56 0)
+			(at 712.47 276.86 0)
 			(hide yes)
 			(show_name no)
@@
 		)
 		(property "Datasheet" ""
-			(at 708.66 289.56 0)
+			(at 712.47 276.86 0)
 			(hide yes)
 			(show_name no)
@@
 		)
 		(property "Description" "Antenna"
-			(at 708.66 289.56 0)
+			(at 712.47 276.86 0)
 			(hide yes)
 			(show_name no)
@@
 	(symbol
 		(lib_id "Device:L")
-		(at 708.66 303.53 0)
+		(at 712.47 290.83 0)
 		(unit 1)
 		(body_style 1)
@@
 		(in_pos_files yes)
 		(dnp no)
-		(fields_autoplaced yes)
 		(property "Reference" "L27"
-			(at 709.93 302.2599 0)
+			(at 712.47 287.274 0)
 			(show_name no)
 			(do_not_autoplace no)
@@
 		)
 		(property "Value" "5.6nH"
-			(at 709.93 304.7999 0)
+			(at 713.74 289.306 0)
 			(show_name no)
 			(do_not_autoplace no)
@@
 		)
 		(property "Footprint" "Inductor_SMD:L_0603_1608Metric_Pad1.05x0.95mm_HandSolder"
-			(at 708.66 303.53 0)
+			(at 712.47 290.83 0)
 			(hide yes)
 			(show_name no)
@@
 		)
 		(property "Datasheet" ""
-			(at 708.66 303.53 0)
+			(at 712.47 290.83 0)
 			(hide yes)
 			(show_name no)
@@
 		)
 		(property "Description" "Inductor"
-			(at 708.66 303.53 0)
+			(at 712.47 290.83 0)
 			(hide yes)
 			(show_name no)
@@
 		(in_pos_files yes)
 		(dnp no)
-		(fields_autoplaced yes)
-		(property "Reference" "FIL1"
-			(at 464.82 66.04 0)
-			(hide yes)
+		(property "Reference" "X1"
+			(at 466.598 72.136 0)
 			(show_name no)
 			(do_not_autoplace no)
@@
 			)
 		)
-		(property "Value" "SF2136E"
-			(at 464.82 66.04 0)
-			(hide yes)
+		(property "Value" "433MHz SAW Filter"
+			(at 474.726 74.168 0)
 			(show_name no)
 			(do_not_autoplace no)
@@
 			(project "Flipper black ki cad"
 				(path "/aadf5baa-c41c-48f9-af5f-e274c89cf282"
-					(reference "FIL1")
+					(reference "X1")
 					(unit 1)
 				)
@@
 	)
 	(symbol
+		(lib_id "Device:C")
+		(at 712.47 300.99 0)
+		(unit 1)
+		(body_style 1)
+		(exclude_from_sim no)
+		(in_bom yes)
+		(on_board yes)
+		(in_pos_files yes)
+		(dnp no)
+		(property "Reference" "C105"
+			(at 715.518 299.72 0)
+			(show_name no)
+			(do_not_autoplace no)
+			(effects
+				(font
+					(size 1.27 1.27)
+				)
+				(justify left)
+			)
+		)
+		(property "Value" "100pf"
+			(at 715.518 302.26 0)
+			(show_name no)
+			(do_not_autoplace no)
+			(effects
+				(font
+					(size 1.27 1.27)
+				)
+				(justify left)
+			)
+		)
+		(property "Footprint" ""
+			(at 713.4352 304.8 0)
+			(hide yes)
+			(show_name no)
+			(do_not_autoplace no)
+			(effects
+				(font
+					(size 1.27 1.27)
+				)
+			)
+		)
+		(property "Datasheet" ""
+			(at 712.47 300.99 0)
+			(hide yes)
+			(show_name no)
+			(do_not_autoplace no)
+			(effects
+				(font
+					(size 1.27 1.27)
+				)
+			)
+		)
+		(property "Description" "Unpolarized capacitor"
+			(at 712.47 300.99 0)
+			(hide yes)
+			(show_name no)
+			(do_not_autoplace no)
+			(effects
+				(font
+					(size 1.27 1.27)
+				)
+			)
+		)
+		(pin "2"
+		)
+		(pin "1"
+		)
+		(instances
+			(project "Flipper black ki cad"
+				(path "/aadf5baa-c41c-48f9-af5f-e274c89cf282"
+					(reference "C105")
+					(unit 1)
+				)
+			)
+		)
+	)
+	(symbol
 		(lib_id "RF_NFC:PN5321A3HN_C1xx")
 		(at 336.55 292.1 0)
@@
 					(unit 1)
 				)
-			)
-		)
-	)
-	(symbol
-		(lib_id "Connector:Barrel_Jack")
-		(at 610.87 293.37 270)
-		(unit 1)
-		(body_style 1)
-		(exclude_from_sim no)
-		(in_bom yes)
-		(on_board yes)
-		(in_pos_files yes)
-		(dnp no)
-		(fields_autoplaced yes)
-		(property "Reference" "J1"
-			(at 615.95 292.0999 90)
-			(show_name no)
-			(do_not_autoplace no)
-			(effects
-				(font
-					(size 1.27 1.27)
-				)
-				(justify left)
-			)
-		)
-		(property "Value" "Barrel_Jack"
-			(at 615.95 294.6399 90)
-			(show_name no)
-			(do_not_autoplace no)
-			(effects
-				(font
-					(size 1.27 1.27)
-				)
-				(justify left)
-			)
-		)
-		(property "Footprint" "Connector_BarrelJack:BarrelJack_Wuerth_694108106102_2.5x5.5mm"
-			(at 609.854 294.64 0)
-			(hide yes)
-			(show_name no)
-			(do_not_autoplace no)
-			(effects
-				(font
-					(size 1.27 1.27)
-				)
-			)
-		)
-		(property "Datasheet" ""
-			(at 609.854 294.64 0)
-			(hide yes)
-			(show_name no)
-			(do_not_autoplace no)
-			(effects
-				(font
-					(size 1.27 1.27)
-				)
-			)
-		)
-		(property "Description" "DC Barrel Jack"
-			(at 610.87 293.37 0)
-			(hide yes)
-			(show_name no)
-			(do_not_autoplace no)
-			(effects
-				(font
-					(size 1.27 1.27)
-				)
-			)
-		)
-		(pin "1"
-		)
-		(pin "2"
-		)
-		(instances
-			(project "Flipper black ki cad"
-				(path "/aadf5baa-c41c-48f9-af5f-e274c89cf282"
-					(reference "J1")
-					(unit 1)
-				)
