File: flipper black PCB/Flipper black ki cad/Flipper black ki cad.kicad_sch (KiCad schematic)
At the start: 246 parts, among them J2 Value: DISP_3.5_WAVESHARE, P1 JST-2pin, P2 USB_C_Plug_USB2.0, Q1 MMBT2222A, Q2 FS8205A, SW1 boot, SW2 REST, SW3 BTN_POWER, SW4 BTN_OK, SW5 BTN_UP, SW6 BTN_DOWN, SW7 BTN_LEFT, SW8 BTN_RIGHT, U1 ESP32-S3, U10 BGA725L6, U11 TLV70018_SOT23-5, U12 TXB0102DCU, U13 MCP23017x-x-SS, U14 TSOP382xx, U15 TP4056, U16 PESD5V0L4UG,115, U17 AP2112K-3.3, U18 DW01A, U2 W25Q128JVS, U3 CC1101, U4 SX1276, U5 PE4259, U6 PE4259, U7 PN5321A3HN, U8 MAX-M8Q, U9 MASW-007221, X1 433MHz SAW Filter, X2 B3715 868MHz SAW Filter, Y1 40MHz SMD 3225, Y2 26 MHz SMD, Y3 32 MHz SMD, Y4 27.120 MHz

Commit message: agg aggg
Parts:
- L10, L9: value 2.7nH -> 47nH
- L11: value 2.7nH -> 23nH
- L5, L6, L7, L8: value 2.7nH -> 27nH
Connections:
- net 12C_SDA: now also U13.13 (SDA)
- net GPS_RXD: no longer TP9.1
- net I2C_SDA: no longer U13.13 (SDA)
- net TOUCH_IRQ: no longer U13.28 (GPA7)
- net TOUCH_RST: now also U13.28 (GPA7)
- net TP_UART_TX: no longer R6.1, U1.49 (U0TXD)
- new net: R6.1, U1.49 (U0TXD)
- new net TP_UART_RX: TP9.1
- no-connect marks 13 -> 20
Changed lines of the file:
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@@
 	)
 	(no_connect
+		(at 331.47 128.27)
+	)
+	(no_connect
+		(at 182.88 100.33)
+	)
+	(no_connect
+		(at 331.47 125.73)
+	)
+	(no_connect
+		(at 331.47 133.35)
+	)
+	(no_connect
 		(at 356.87 287.02)
 	)
@@
 	)
 	(no_connect
+		(at 331.47 130.81)
+	)
+	(no_connect
 		(at 356.87 289.56)
 	)
 	(no_connect
+		(at 182.88 102.87)
+	)
+	(no_connect
 		(at 316.23 271.78)
 	)
@@
 	)
 	(no_connect
+		(at 331.47 123.19)
+	)
+	(no_connect
 		(at 316.23 294.64)
 	)
@@
 	(wire
 		(pts
-			(xy 151.13 138.43) (xy 182.88 138.43)
-		)
-		(stroke
-			(width 0)
-			(type default)
-		)
-	)
-	(wire
-		(pts
 			(xy 431.8 416.56) (xy 431.8 412.75)
 		)
@@
 	(wire
 		(pts
-			(xy 284.48 386.08) (xy 264.16 386.08)
+			(xy 284.48 386.08) (xy 271.78 386.08)
 		)
 		(stroke
@@
 	(wire
 		(pts
+			(xy 151.13 138.43) (xy 182.88 138.43)
+		)
+		(stroke
+			(width 0)
+			(type default)
+		)
+	)
+	(wire
+		(pts
 			(xy 251.46 410.21) (xy 251.46 420.37)
 		)
@@
 	(wire
 		(pts
-			(xy 264.16 386.08) (xy 264.16 381)
+			(xy 271.78 386.08) (xy 271.78 381)
 		)
 		(stroke
@@
 	(wire
 		(pts
-			(xy 264.16 381) (xy 272.796 381)
+			(xy 271.78 381) (xy 272.796 381)
 		)
 		(stroke
@@
 		)
 	)
-	(global_label "TP_UART_TX"
-		(shape input)
-		(at 151.13 135.89 0)
-		(fields_autoplaced yes)
-		(effects
-			(font
-				(size 1.27 1.27)
-				(thickness 0.1588)
-			)
-			(justify left)
-		)
-		(property "Intersheetrefs" "${INTERSHEET_REFS}"
-			(at 165.1218 135.89 0)
-			(hide yes)
-			(show_name no)
-			(do_not_autoplace no)
-			(effects
-				(font
-					(size 1.27 1.27)
-				)
-				(justify left)
-			)
-		)
-	)
 	(global_label "BTN_UP"
 		(shape input)
@@
 		)
 	)
-	(global_label "I2C_SDA"
-		(shape input)
-		(at 774.7 120.65 180)
-		(fields_autoplaced yes)
-		(effects
-			(font
-				(size 1.27 1.27)
-			)
-			(justify right)
-		)
-		(property "Intersheetrefs" "${INTERSHEET_REFS}"
-			(at 764.0948 120.65 0)
-			(hide yes)
-			(show_name no)
-			(do_not_autoplace no)
-			(effects
-				(font
-					(size 1.27 1.27)
-				)
-				(justify right)
-			)
-		)
-	)
 	(global_label "DISP_BL"
 		(shape input)
@@
 		)
 	)
-	(global_label "TP_UART_RX"
-		(shape input)
-		(at 151.13 138.43 0)
-		(fields_autoplaced yes)
-		(effects
-			(font
-				(size 1.27 1.27)
-				(thickness 0.1588)
-			)
-			(justify left)
-		)
-		(property "Intersheetrefs" "${INTERSHEET_REFS}"
-			(at 165.4242 138.43 0)
-			(hide yes)
-			(show_name no)
-			(do_not_autoplace no)
-			(effects
-				(font
-					(size 1.27 1.27)
-				)
-				(justify left)
-			)
-		)
-	)
 	(global_label "BTN_POWER"
 		(shape input)
@@
 		)
 	)
-	(global_label "TOUCH_IRQ"
+	(global_label "GPS_EXTINT"
 		(shape input)
-		(at 800.1 135.89 0)
+		(at 510.54 300.99 180)
 		(fields_autoplaced yes)
 		(effects
@@
 				(thickness 0.1588)
 			)
-			(justify left)
+			(justify right)
 		)
 		(property "Intersheetrefs" "${INTERSHEET_REFS}"
-			(at 813.4872 135.89 0)
+			(at 496.6087 300.99 0)
 			(hide yes)
 			(show_name no)
@@
 					(size 1.27 1.27)
 				)
-				(justify left)
+				(justify right)
 			)
 		)
 	)
-	(global_label "GPS_EXTINT"
+	(global_label "CS_SX1276"
 		(shape input)
-		(at 510.54 300.99 180)
+		(at 182.88 110.49 0)
 		(fields_autoplaced yes)
 		(effects
@@
 				(thickness 0.1588)
 			)
-			(justify right)
+			(justify left)
 		)
 		(property "Intersheetrefs" "${INTERSHEET_REFS}"
-			(at 496.6087 300.99 0)
+			(at 196.5693 110.49 0)
 			(hide yes)
 			(show_name no)
@@
 					(size 1.27 1.27)
 				)
-				(justify right)
+				(justify left)
 			)
 		)
 	)
-	(global_label "CS_SX1276"
+	(global_label "TOUCH_RST"
 		(shape input)
-		(at 182.88 110.49 0)
+		(at 800.1 135.89 0)
 		(fields_autoplaced yes)
 		(effects
@@
 		)
 		(property "Intersheetrefs" "${INTERSHEET_REFS}"
-			(at 196.5693 110.49 0)
+			(at 813.729 135.89 0)
 			(hide yes)
 			(show_name no)
@@
 		)
 	)
+	(global_label "12C_SDA"
+		(shape input)
+		(at 774.7 120.65 180)
+		(fields_autoplaced yes)
+		(effects
+			(font
+				(size 1.27 1.27)
+				(thickness 0.1588)
+			)
+			(justify right)
+		)
+		(property "Intersheetrefs" "${INTERSHEET_REFS}"
+			(at 763.4901 120.65 0)
+			(hide yes)
+			(show_name no)
+			(do_not_autoplace no)
+			(effects
+				(font
+					(size 1.27 1.27)
+				)
+				(justify right)
+			)
+		)
+	)
 	(global_label "IR_TX"
 		(shape input)
@@
 			)
 		)
-		(property "Value" "2.7nH"
+		(property "Value" "47nH"
 			(at 181.61 277.368 90)
 			(show_name no)
@@
 			)
 		)
-		(property "Value" "2.7nH"
+		(property "Value" "27nH"
 			(at 130.81 283.718 90)
 			(show_name no)
@@
 			)
 		)
-		(property "Value" "2.7nH"
+		(property "Value" "27nH"
 			(at 130.81 271.018 90)
 			(show_name no)
@@
 			)
 		)
-		(property "Value" "2.7nH"
+		(property "Value" "27nH"
 			(at 154.94 271.018 90)
 			(show_name no)
@@
 			)
 		)
-		(property "Value" "2.7nH"
+		(property "Value" "27nH"
 			(at 143.256 291.846 0)
 			(show_name no)
@@
 			)
 		)
-		(property "Value" "2.7nH"
+		(property "Value" "23nH"
 			(at 212.344 290.068 90)
 			(show_name no)
@@
 			)
 		)
-		(property "Value" "2.7nH"
+		(property "Value" "47nH"
 			(at 168.91 277.368 90)
 			(show_name no)

Commit message: fahh
Parts:
- added C106: 10uf, symbol Device:C
- added C107: 100nf, symbol Device:C
Connections:
- net GND: now also C106.2, C107.2
- net VDD33: now also C106.1, C107.1

Commit message: rthniew
Parts:
- added FB2: BLM21PG221SN1D, Inductor_SMD:L_0603_1608Metric_Pad1.05x0.95mm_HandSolder, symbol Device:FerriteBead
- added R45: 10k, Resistor_SMD:R_0402_1005Metric, symbol Device:R
- FB1: value FerriteBead -> BLM21PG221SN1D
Connections:
- net GND: now also FB2.2; no longer P2.SH (SHIELD)
- net VDD33: now also R45.1; no longer U13.18 (~{RESET})
- new net: FB2.1, P2.SH (SHIELD)
- new net: R45.2, U13.18 (~{RESET})
Other:
- moved on the sheet: D4

Commit message: fahh
Parts:
- C105, C106, C107: footprint (none) -> Capacitor_SMD:C_0603_1608Metric_Pad1.08x0.95mm_HandSolder
Changed lines of the file:
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@@
 			)
 		)
-		(property "Footprint" ""
+		(property "Footprint" "Capacitor_SMD:C_0603_1608Metric_Pad1.08x0.95mm_HandSolder"
 			(at 780.7452 99.06 0)
 			(hide yes)
@@
 			)
 		)
-		(property "Footprint" ""
+		(property "Footprint" "Capacitor_SMD:C_0603_1608Metric_Pad1.08x0.95mm_HandSolder"
 			(at 768.0452 99.06 0)
 			(hide yes)
@@
 			)
 		)
-		(property "Footprint" ""
+		(property "Footprint" "Capacitor_SMD:C_0603_1608Metric_Pad1.08x0.95mm_HandSolder"
 			(at 713.4352 304.8 0)
 			(hide yes)

Commit message: uubbj
Parts:
- P1: footprint Connector_JST:JST_EH_S3B-EH_1x03_P2.50mm_Horizontal -> Connector_JST:JST_PH_S2B-PH-SM4-TB_1x02-1MP_P2.00mm_Horizontal
- Q2: footprint SOP65P640X120-8N -> FS8205A:SOP65P640X120-8N
- SW3, SW4, SW5, SW6, SW7, SW8: footprint Button_Switch_SMD:SW_DIP_SPSTx01_Slide_6.7x4.1mm_W6.73mm_P2.54mm_LowProfile_JPin -> PTS645SH43SMTR92LFS buttons:SW_PTS645SH43SMTR92LFS
- TP1, TP10, TP2, TP3, TP4, TP5, TP7, TP8, TP9: footprint TestPoint:TestPoint_2Pads_Pitch2.54mm_Drill0.8mm -> TestPoint:TestPoint_Pad_D1.0mm
- U16: footprint SOT65P210X110-5N -> PESD5V0L4UG_115:SOT65P210X110-5N
- U3: footprint QLP20 -> CC1101 real:QLP20
- U5, U6: footprint SOT65P215X110-6N -> PE4259:SOT65P215X110-6N
- X1: footprint RFM-SAW-3X3MM -> SF2136E:RFM-SAW-3X3MM
Changed lines of the file:
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@@
 			)
 		)
-		(property "Footprint" "TestPoint:TestPoint_2Pads_Pitch2.54mm_Drill0.8mm"
+		(property "Footprint" "TestPoint:TestPoint_Pad_D1.0mm"
 			(at 690.88 408.94 0)
 			(hide yes)
@@
 			)
 		)
-		(property "Footprint" "TestPoint:TestPoint_2Pads_Pitch2.54mm_Drill0.8mm"
+		(property "Footprint" "TestPoint:TestPoint_Pad_D1.0mm"
 			(at 741.68 375.92 0)
 			(hide yes)
@@
 			)
 		)
-		(property "Footprint" "Button_Switch_SMD:SW_DIP_SPSTx01_Slide_6.7x4.1mm_W6.73mm_P2.54mm_LowProfile_JPin"
+		(property "Footprint" "PTS645SH43SMTR92LFS buttons:SW_PTS645SH43SMTR92LFS"
 			(at 588.01 396.24 0)
 			(hide yes)
@@
 			)
 		)
-		(property "Footprint" "SOT65P210X110-5N"
+		(property "Footprint" "PESD5V0L4UG_115:SOT65P210X110-5N"
 			(at 487.68 419.1 0)
 			(hide yes)
@@
 			)
 		)
-		(property "Footprint" "TestPoint:TestPoint_2Pads_Pitch2.54mm_Drill0.8mm"
+		(property "Footprint" "TestPoint:TestPoint_Pad_D1.0mm"
 			(at 767.08 408.94 0)
 			(hide yes)
@@
 			)
 		)
-		(property "Footprint" "Button_Switch_SMD:SW_DIP_SPSTx01_Slide_6.7x4.1mm_W6.73mm_P2.54mm_LowProfile_JPin"
+		(property "Footprint" "PTS645SH43SMTR92LFS buttons:SW_PTS645SH43SMTR92LFS"
 			(at 636.27 397.51 0)
 			(hide yes)
@@
 			)
 		)
-		(property "Footprint" "Button_Switch_SMD:SW_DIP_SPSTx01_Slide_6.7x4.1mm_W6.73mm_P2.54mm_LowProfile_JPin"
+		(property "Footprint" "PTS645SH43SMTR92LFS buttons:SW_PTS645SH43SMTR92LFS"
 			(at 544.83 368.3 0)
 			(hide yes)
@@
 			)
 		)
-		(property "Footprint" "Button_Switch_SMD:SW_DIP_SPSTx01_Slide_6.7x4.1mm_W6.73mm_P2.54mm_LowProfile_JPin"
+		(property "Footprint" "PTS645SH43SMTR92LFS buttons:SW_PTS645SH43SMTR92LFS"
 			(at 544.83 396.24 0)
 			(hide yes)
@@
 			)
 		)
-		(property "Footprint" "Button_Switch_SMD:SW_DIP_SPSTx01_Slide_6.7x4.1mm_W6.73mm_P2.54mm_LowProfile_JPin"
+		(property "Footprint" "PTS645SH43SMTR92LFS buttons:SW_PTS645SH43SMTR92LFS"
 			(at 636.27 369.57 0)
 			(hide yes)
@@
 			)
 		)
-		(property "Footprint" "TestPoint:TestPoint_2Pads_Pitch2.54mm_Drill0.8mm"
+		(property "Footprint" "TestPoint:TestPoint_Pad_D1.0mm"
 			(at 716.28 408.94 0)
 			(hide yes)
@@
 			)
 		)
-		(property "Footprint" "RFM-SAW-3X3MM"
+		(property "Footprint" "SF2136E:RFM-SAW-3X3MM"
 			(at 464.566 69.85 0)
 			(hide yes)
@@
 			)
 		)
-		(property "Footprint" "SOT65P215X110-6N"
+		(property "Footprint" "PE4259:SOT65P215X110-6N"
 			(at 552.45 72.39 0)
 			(hide yes)
@@
 			)
 		)
-		(property "Footprint" "SOT65P215X110-6N"
+		(property "Footprint" "PE4259:SOT65P215X110-6N"
 			(at 551.18 163.83 0)
 			(hide yes)
@@
 			)
 		)
-		(property "Footprint" "TestPoint:TestPoint_2Pads_Pitch2.54mm_Drill0.8mm"
+		(property "Footprint" "TestPoint:TestPoint_Pad_D1.0mm"
 			(at 741.68 408.94 0)
 			(hide yes)
@@
 			)
 		)
-		(property "Footprint" "TestPoint:TestPoint_2Pads_Pitch2.54mm_Drill0.8mm"
+		(property "Footprint" "TestPoint:TestPoint_Pad_D1.0mm"
 			(at 690.88 375.92 0)
 			(hide yes)
@@
 			)
 		)
-		(property "Footprint" "SOP65P640X120-8N"
+		(property "Footprint" "FS8205A:SOP65P640X120-8N"
 			(at 269.24 420.37 0)
 			(hide yes)
@@
 			)
 		)
-		(property "Footprint" "TestPoint:TestPoint_2Pads_Pitch2.54mm_Drill0.8mm"
+		(property "Footprint" "TestPoint:TestPoint_Pad_D1.0mm"
 			(at 767.08 375.92 0)
 			(hide yes)
@@
 			)
 		)
-		(property "Footprint" "Connector_JST:JST_EH_S3B-EH_1x03_P2.50mm_Horizontal"
+		(property "Footprint" "Connector_JST:JST_PH_S2B-PH-SM4-TB_1x02-1MP_P2.00mm_Horizontal"
 			(at 281.94 379.73 0)
 			(hide yes)
@@
 			)
 		)
-		(property "Footprint" "TestPoint:TestPoint_2Pads_Pitch2.54mm_Drill0.8mm"
+		(property "Footprint" "TestPoint:TestPoint_Pad_D1.0mm"
 			(at 716.28 375.92 0)
 			(hide yes)
@@
 			)
 		)
-		(property "Footprint" "Button_Switch_SMD:SW_DIP_SPSTx01_Slide_6.7x4.1mm_W6.73mm_P2.54mm_LowProfile_JPin"
+		(property "Footprint" "PTS645SH43SMTR92LFS buttons:SW_PTS645SH43SMTR92LFS"
 			(at 588.01 368.3 0)
 			(hide yes)
@@
 			)
 		)
-		(property "Footprint" "TestPoint:TestPoint_2Pads_Pitch2.54mm_Drill0.8mm"
+		(property "Footprint" "TestPoint:TestPoint_Pad_D1.0mm"
 			(at 792.48 375.92 0)
 			(hide yes)
@@
 			)
 		)
-		(property "Footprint" "QLP20"
+		(property "Footprint" "CC1101 real:QLP20"
 			(at 59.69 275.59 0)
 			(hide yes)

Commit message: yooo
Parts:
- added C108: 1uf, symbol Device:C
- added C109: 100nf, symbol Device:C
- added U19: SX1262IMLTRT, Package_DFN_QFN:QFN-24-1EP_4x4mm_P0.5mm_EP2.6x2.6mm, symbol RF:SX1262IMLTRT
- added Y5: 32 MHz SMD, Crystal:Crystal_SMD_2016-4Pin_2.0x1.6mm, symbol Device:Crystal
Connections:
- net CS_SX1276: now also U19.19 (NSS)
- net GND: now also C108.2, C109.2
- net SPI_MISO: now also U19.16 (MISO)
- net SPI_MOSI: now also U19.17 (MOSI)
- net SPI_SCK: now also U19.18 (SCK)
- net VDD33: now also C108.1, C109.1, U19.1 (VDD_IN), U19.10 (VBAT), U19.11 (VBAT_IO)
- new net: U19.4 (XTB), Y5.1
- new net: U19.3 (XTA), Y5.2
- no-connect marks 20 -> 23

Commit message: yooo
Parts:
- removed C29, C30, C31, C32, C33, C34, C57: 100nf, Capacitor_SMD:C_0603_1608Metric_Pad1.08x0.95mm_HandSolder, symbol Device:C
- removed C35, C36: 15pf, Capacitor_SMD:C_0603_1608Metric_Pad1.08x0.95mm_HandSolder, symbol Device:C
- removed C37, C38, C39, C40, C41, C42, C43, C44, C45, C46: 3.3pf, Capacitor_SMD:C_0603_1608Metric_Pad1.08x0.95mm_HandSolder, symbol Device:C
- removed C47, C48, C61, C62: 1nf, Capacitor_SMD:C_0603_1608Metric_Pad1.08x0.95mm_HandSolder, symbol Device:C
- removed C49, C50, C51, C58: 2.2pf, Capacitor_SMD:C_0603_1608Metric_Pad1.08x0.95mm_HandSolder, symbol Device:C
- removed C52, C54, C64, C65: 1.8pf, Capacitor_SMD:C_0603_1608Metric_Pad1.08x0.95mm_HandSolder, symbol Device:C
- removed C53, C55, C56, C60: 1.5pf, Capacitor_SMD:C_0603_1608Metric_Pad1.08x0.95mm_HandSolder, symbol Device:C
- removed C59: 1.0pf, Capacitor_SMD:C_0603_1608Metric_Pad1.08x0.95mm_HandSolder, symbol Device:C
- removed C63: 1.5 pf, Capacitor_SMD:C_0603_1608Metric_Pad1.08x0.95mm_HandSolder, symbol Device:C
- removed C66: 1uF, Capacitor_SMD:C_0603_1608Metric_Pad1.08x0.95mm_HandSolder, symbol Device:C
- removed L12: 24nH, Inductor_SMD:L_0603_1608Metric_Pad1.05x0.95mm_HandSolder, symbol Device:L
- removed L13, L14, L24: 100nH, Inductor_SMD:L_0603_1608Metric_Pad1.05x0.95mm_HandSolder, symbol Device:L
- removed L15, L16, L17, L20: 120nH, Inductor_SMD:L_0603_1608Metric_Pad1.05x0.95mm_HandSolder, symbol Device:L
- removed L18, L19: 68nH, Inductor_SMD:L_0603_1608Metric_Pad1.05x0.95mm_HandSolder, symbol Device:L
- removed L21, L22, L23: 22nH, Inductor_SMD:L_0603_1608Metric_Pad1.05x0.95mm_HandSolder, symbol Device:L
- removed R10, R11, R12, R13, R14, R16, R8, R9: 0R, Resistor_SMD:R_0402_1005Metric, symbol Device:R
- removed R15: 1k, Resistor_SMD:R_0402_1005Metric, symbol Device:R
- removed R17: 10k, Resistor_SMD:R_0402_1005Metric, symbol Device:R
- removed SX1276, SX1276_1: 50ohm, Connector_Coaxial:U.FL_Hirose_U.FL-R-SMT-1_Vertical, symbol Device:Antenna
- removed U4: SX1276, Package_DFN_QFN:QFN-28-1EP_6x6mm_P0.65mm_EP4.8x4.8mm, symbol RF:SX1276
- removed U5, U6: PE4259, PE4259:SOT65P215X110-6N, symbol PE4259:PE4259
- removed X1: 433MHz SAW Filter, SF2136E:RFM-SAW-3X3MM, symbol SF2136E:SF2136E
- removed X2: B3715 868MHz SAW Filter, Filter:Filter_SAW_Epcos_DCC6C_3x3mm, symbol RF_Filter:B3715
- removed Y3: 32 MHz SMD, Crystal:Crystal_SMD_2016-4Pin_2.0x1.6mm, symbol Device:Crystal
- added C110: 470nf, Capacitor_SMD:C_0603_1608Metric_Pad1.08x0.95mm_HandSolder, symbol Device:C
- added C111, C112, C118, C120, C123: 10pf, Capacitor_SMD:C_0603_1608Metric_Pad1.08x0.95mm_HandSolder, symbol Device:C
- added C113, C121: 100nf, Capacitor_SMD:C_0603_1608Metric_Pad1.08x0.95mm_HandSolder, symbol Device:C
- added C114: 6.8pf, Capacitor_SMD:C_0603_1608Metric_Pad1.08x0.95mm_HandSolder, symbol Device:C
- added C115, C125: 8.2pf, Capacitor_SMD:C_0603_1608Metric_Pad1.08x0.95mm_HandSolder, symbol Device:C
- added C116, C122: 1nf, Capacitor_SMD:C_0603_1608Metric_Pad1.08x0.95mm_HandSolder, symbol Device:C
- added C117, C124: 5.6pf, Capacitor_SMD:C_0603_1608Metric_Pad1.08x0.95mm_HandSolder, symbol Device:C
- added C119: 22pf, Capacitor_SMD:C_0603_1608Metric_Pad1.08x0.95mm_HandSolder, symbol Device:C
- added L28, L33: 18nH, Inductor_SMD:L_0603_1608Metric_Pad1.05x0.95mm_HandSolder, symbol Device:L
- added L29, L30: 15nH, Inductor_SMD:L_0603_1608Metric_Pad1.05x0.95mm_HandSolder, symbol Device:L
- added L31, L34: 22nH, Inductor_SMD:L_0603_1608Metric_Pad1.05x0.95mm_HandSolder, symbol Device:L
- added L32: 27nH, Inductor_SMD:L_0603_1608Metric_Pad1.05x0.95mm_HandSolder, symbol Device:L
- added R46: 10k, Resistor_SMD:R_0402_1005Metric, symbol Device:R
- added R47, R48: 100R, Resistor_SMD:R_0402_1005Metric, symbol Device:R
- added SX1262: 50ohm, Connector_Coaxial:U.FL_Hirose_U.FL-R-SMT-1_Vertical, symbol Device:Antenna
- added U20: PE4259, PE4259:SOT65P215X110-6N, symbol PE4259:PE4259
- C108, C109: footprint (none) -> Capacitor_SMD:C_0603_1608Metric_Pad1.08x0.95mm_HandSolder
- P2: footprint Connector_USB:USB_C_Receptacle_XKB_U262-16XN-4BVC11 -> Connector_USB:USB_C_Receptacle_GCT_USB4105-xx-A_16P_TopMnt_Horizontal
- U19: footprint Package_DFN_QFN:QFN-24-1EP_4x4mm_P0.5mm_EP2.6x2.6mm -> SX1262IMLTRT:QFN50P400X400X100-25N
Connections:
- net SPID is gone; now on net SX1262_DIO2: R2.2
- net SPIQ is gone; now on net SX1262_BUSY: R1.2
- net SX1276_DIO0 is gone; now on net SX1262_DIO1: U1.44 (MTCK)
- net SX1276_RESET is gone; now on net SX1262_RESET: U1.45 (MTDO)
- net TP_UART_RX is gone; now on net GPS_RXD: TP9.1
- net GND: now also U19.2 (GND), U19.20 (GND), U19.25 (GND), U19.5 (GND), U19.8 (GND), C110.2, C111.2, C112.2, C114.2, C115.2, C116.2, C118.2, C120.1, C121.1, C122.2, C124.1, C125.1, U20.2 (GND)
- net TP_UART_TX: now also R6.1, U1.49 (U0TXD)
- net VDD33: now also R46.2, R47.1
- net SX1262_DIO2: now reaches U19.12 (DIO2)
- net SX1262_DIO2: now also R48.1
- net SX1262_DIO1: now reaches U19.13 (DIO1)
- net SX1262_BUSY: now reaches U19.14 (BUSY)
- net SX1262_RESET: now reaches U19.15 (~{RESET})
- net SX1262_RESET: now also R46.1
- net at U19.21 (RFI_P): now also C121.2, L33.1
- net at U19.22 (RFI_N): now also C119.1, L33.2
- net at U19.23 (RFO): now also L30.1
- net at U19.24 (VR_PA): now also C111.1, C112.1, L29.2
- net at U19.7 (VREG): now also C110.1, L28.2
- net at U19.9 (DCC_SW): now also L28.1
- net CS_SX1276 renamed CS_SX1262
- new net: C119.2, C120.2, U20.3 (RF2)
- new net: C123.2, C124.2, L34.1
- new net: C125.2, L34.2, SX1262.1 (A)
- new net: C122.1, R48.2, U20.4 (CTRL)
- new net: C113.1, C114.1, L29.1, L30.2, L31.1
- new net: C113.2, C115.1, C117.1, L31.2
- new net: C123.1, U20.5 (RFC)
- new net: C117.2, L32.1
- new net: C116.1, R47.2, U20.6 (~{CTRL/}VDD)
- new net: C118.1, L32.2, U20.1 (RF1)
- no-connect marks 23 -> 13
Other:
- note added: "SX1262 - LoRa Transceiver"
- note removed: "RF Switch HF"
- note removed: "SX1276 - LoRa Transceiver"
- moved on the sheet: C108, C109, U19, Y5

Commit message: fie
Parts:
- PN532_ANT1: footprint ESP_Antenna:ESPRESSIF_ESP32_MIFA_2.4GHz_Right -> NFC_ANTENNA:NFC_ANT
- R6: value 499Ohm -> 499R
- renumbered R_RSTPD1 to R_38, R_GPIO45 to R_G45, R_GPIO46 to R_G46
Other:
- moved on the sheet: C108, C109, C110, C111, C112, C113, C114, C115, C116, C117, C118, C119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
