File: flipper black PCB/Flipper black ki cad/Flipper black ki cad.kicad_pcb (KiCad board)
At the start: 4 copper layers, 305 x 146.4 mm, 213 parts, among them J2 Value: DISP_3.5_WAVESHARE, P1 JST-2pin, P2 USB_C_Plug_USB2.0, Q1 MMBT2222A, Q2 FS8205A, SW1 boot, SW2 REST, SW3 BTN_POWER, SW4 BTN_OK, SW5 BTN_UP, SW6 BTN_DOWN, SW7 BTN_LEFT, SW8 BTN_RIGHT, U1 ESP32-S3, U10 BGA725L6, U11 TLV70018_SOT23-5, U12 TXB0102DCU, U13 MCP23017x-x-SS, U14 TSOP382xx, U15 TP4056, U16 PESD5V0L4UG,115, U17 AP2112K-3.3, U18 DW01A, U19 SX1262IMLTRT, U2 W25Q128JVS, U20 PE4259, U3 CC1101, U7 PN5321A3HN, U8 MAX-M8Q, U9 MASW-007221, Y1 40MHz SMD 3225, Y2 26 MHz SMD, Y4 27.120 MHz, Y5 32 MHz SMD

Commit message: zeeha
Parts:
- moved GPS_ANT1 282.5 mm to (166.1, 71.5)
- moved PCB_ANT1 238.2 mm to (179.4, 71.5)
- moved SX1262 210.5 mm to (218.2, 71.5)
- moved PN532_ANT1 183.1 mm to (193.3, 74.8)
- moved C67 124.6 mm to (164.8, 83.5)
- moved C69 124.6 mm to (160.3, 89.4)
- moved C73 124.6 mm to (170.3, 95.0)
- moved C74 124.6 mm to (173.1, 95.0)
- moved C75 124.6 mm to (169.6, 82.5)
- moved C77 124.6 mm to (177.2, 87.5)
- moved C78 124.6 mm to (175.9, 80.8)
- moved C79 124.6 mm to (177.3, 91.4)
- moved C80 124.6 mm to (179.7, 83.8)
- moved C82 124.6 mm to (167.6, 95.0)
- moved C83 124.6 mm to (165.1, 95.0)
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Other:
- board size 305 x 146.4 mm -> 92.3 x 143 mm

Commit message: yaya
Parts:
- moved IR_LEDs1 2.01 mm to (182.5, 140.0)
- moved IR_LEDs2 2.01 mm to (189.3, 140.0)
- moved IR_LEDs3 2.01 mm to (196.1, 140.0)
- moved PN532_ANT1 0.73 mm to (193.4, 75.5)
- moved J2 0.62 mm to (198.0, 72.1)
Routing:
- net GND: track 0.00 -> 109.6 mm, vias 0 -> 127
- added copper zone on In1.Cu, net GND
