File: flipper black PCB/Flipper black ki cad/Flipper black ki cad.kicad_pcb (KiCad board)
At the start: 4 copper layers, 92.3 x 143 mm, 213 parts, among them J2 Value: DISP_3.5_WAVESHARE, P1 JST-2pin, P2 USB_C_Plug_USB2.0, Q1 MMBT2222A, Q2 FS8205A, SW1 boot, SW2 REST, SW3 BTN_POWER, SW4 BTN_OK, SW5 BTN_UP, SW6 BTN_DOWN, SW7 BTN_LEFT, SW8 BTN_RIGHT, U1 ESP32-S3, U10 BGA725L6, U11 TLV70018_SOT23-5, U12 TXB0102DCU, U13 MCP23017x-x-SS, U14 TSOP382xx, U15 TP4056, U16 PESD5V0L4UG,115, U17 AP2112K-3.3, U18 DW01A, U19 SX1262IMLTRT, U2 W25Q128JVS, U20 PE4259, U3 CC1101, U7 PN5321A3HN, U8 MAX-M8Q, U9 MASW-007221, Y1 40MHz SMD 3225, Y2 26 MHz SMD, Y4 27.120 MHz, Y5 32 MHz SMD

Commit message: yay
Parts:
- removed PN532_ANT1: 50ohm, NFC_ANTENNA:NFC_ANT
- added AE1: Antenna_Loop, KiCad_Package coil:NFC_45x45_N4_NXP_PN5180, B.Cu at (198.4, 106.8)
Connections:
- C78 pad 2: GND -> Net-(AE1-Pad1)
- C79 pad 2: GND -> Net-(AE1-Pad1)
- C80 pad 2: GND -> Net-(AE1-Pad2)
- C81 pad 1: GND -> Net-(AE1-Pad2)
Routing:
- net Net-(AE1-Pad1): track 0.00 -> 15.7 mm, vias 0 -> 3
- net Net-(AE1-Pad2): track 0.00 -> 13.3 mm, vias 0 -> 3
- net GND: track 110.2 -> 106.6 mm, vias 127 -> 123

Commit message: u
Routing:
- net PN532_RESET: track 0.00 -> 58.6 mm
- net PN532_IRQ: track 0.00 -> 49.4 mm, vias 0 -> 2
- net GPS_EXTINT: track 0.00 -> 49.2 mm, vias 0 -> 2
- net CS_PN532: track 0.00 -> 45.7 mm, vias 0 -> 2

Commit message: kdhe
Parts:
- moved R5 1.23 mm to (209.6, 112.0)
- moved R4 0.23 mm to (209.6, 108.5)
Routing:
- net SPI_SCK: track 0.00 -> 129.2 mm, vias 0 -> 6
- net SPI_MISO: track 0.00 -> 125.8 mm, vias 0 -> 9
- net SPI_MOSI: track 0.00 -> 123.1 mm, vias 0 -> 11
- net USB_DN: track 0.00 -> 87.4 mm, vias 0 -> 2
- net USB_DP: track 0.00 -> 86.0 mm, vias 0 -> 2
- net DISP_MISO: track 0.00 -> 54.2 mm, vias 0 -> 3
- net GPS_TIMEPULSE: track 0.00 -> 46.2 mm, vias 0 -> 2
- net I2C_SCL: track 0.00 -> 40.8 mm, vias 0 -> 3
- net CS_SX1262: track 0.00 -> 31.0 mm
- net BTN_POWER: track 0.00 -> 30.2 mm
- net Net-(U1-SPIQ): track 0.00 -> 14.2 mm, vias 0 -> 2
- net Net-(U1-SPICLK): track 0.00 -> 12.7 mm, vias 0 -> 2
- net Net-(U1-SPID): track 0.00 -> 8.59 mm, vias 0 -> 2
- net Net-(Q2-~-Pad1): track 0.00 -> 5.76 mm
- net Net-(U1-SPIHD): track 0.00 -> 4.69 mm
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
Commit message: fajhh
Routing:
- net EN_BTN: track 0.00 -> 145.9 mm, vias 0 -> 10
- net BOOT_BTN: track 0.00 -> 130.7 mm, vias 0 -> 10
- net BTN_OK: track 0.00 -> 72.9 mm, vias 0 -> 6
- net BTN_UP: track 0.00 -> 69.0 mm, vias 0 -> 4
- net BTN_DOWN: track 0.00 -> 68.8 mm, vias 0 -> 2
- net CS_CC1101: track 0.00 -> 65.0 mm, vias 0 -> 2
- net CC1101_GDO0: track 0.00 -> 61.3 mm, vias 0 -> 4
- net CC1101_GDO2: track 0.00 -> 49.8 mm, vias 0 -> 2
- net GPS_RESET: track 0.00 -> 41.2 mm, vias 0 -> 2
- net GPS_SCL: track 0.00 -> 38.1 mm, vias 0 -> 2
- net GPS_SDA: track 0.00 -> 35.6 mm, vias 0 -> 4
- net FLASH_IO3: track 0.00 -> 35.5 mm, vias 0 -> 4
- net FLASH_IO0: track 0.00 -> 28.4 mm, vias 0 -> 6
- net FLASH_CLK: track 0.00 -> 23.1 mm, vias 0 -> 2
- net FLASH_IO2: track 0.00 -> 17.9 mm, vias 0 -> 4
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
Commit message: hell
Parts:
- moved L2 0.27 mm to (202.6, 98.5)
- moved L4 0.27 mm to (198.6, 98.5)
Routing:
- net Net-(U1-LNA_IN): track 0.00 -> 33.4 mm, vias 0 -> 4
- net Net-(C3-Pad1): track 0.40 -> 28.1 mm, vias 0 -> 4
- net Net-(U1-XTAL_P): track 0.00 -> 10.9 mm, vias 0 -> 2
- net EN_BTN: track 145.9 -> 147.2 mm
- net BOOT_BTN: track 130.7 -> 131.5 mm
- net BTN_UP: track 69.0 -> 69.7 mm
- net GPS_RESET: track 41.2 -> 40.5 mm
- net CC1101_GDO2: track 49.8 -> 50.4 mm
- net GPS_EXTINT: track 50.1 -> 49.5 mm

Commit message: rt
Parts:
- AE1: value Antenna_Loop -> PN532 ANT
- L25, L26: value 560nH -> 220nH
- moved C25 106.5 mm to (151.4, 141.2)
- moved C26 106.5 mm to (144.4, 147.2)
- moved C28 106.5 mm to (133.4, 146.8)
- moved C18 106.5 mm to (139.2, 143.8)
- moved C20 106.5 mm to (129.8, 137.6)
- moved C21 106.5 mm to (135.8, 143.8)
- moved C22 106.5 mm to (147.8, 144.8)
- moved C23 106.5 mm to (137.1, 146.8)
- moved C24 106.5 mm to (144.1, 144.8)
- moved C27 106.5 mm to (141.2, 145.1)
- moved L10 106.5 mm to (151.2, 137.6)
- moved L11 106.5 mm to (142.8, 141.6)
- moved L5 106.5 mm to (142.8, 137.6)
- moved L6 106.5 mm to (145.8, 137.6)
- moved L7 106.5 mm to (148.8, 137.6)
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Routing:
- net EN_BTN: track 147.2 -> 0.00 mm, vias 10 -> 0
- net BOOT_BTN: track 131.5 -> 0.00 mm, vias 10 -> 0
- net SPI_SCK: track 129.9 -> 0.00 mm, vias 6 -> 0
- net SPI_MISO: track 129.3 -> 0.00 mm, vias 9 -> 0
- net SPI_MOSI: track 125.8 -> 0.00 mm, vias 11 -> 0
- net GND: track 106.6 -> 0.00 mm, vias 123 -> 0
- net USB_DN: track 89.3 -> 0.00 mm, vias 2 -> 0
- net USB_DP: track 87.4 -> 0.00 mm, vias 2 -> 0
- net BTN_OK: track 72.8 -> 0.00 mm, vias 6 -> 0
- net BTN_UP: track 69.7 -> 0.00 mm, vias 4 -> 0
- net BTN_DOWN: track 68.8 -> 0.00 mm, vias 2 -> 0
- net CS_CC1101: track 65.0 -> 0.00 mm, vias 2 -> 0
- net PN532_RESET: track 63.8 -> 0.00 mm
- net CC1101_GDO0: track 61.7 -> 0.00 mm, vias 4 -> 0
- net VDD33: track 56.3 -> 0.00 mm, vias 70 -> 0
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