File: flipper black PCB/Flipper black ki cad/Flipper black ki cad.kicad_pcb (KiCad board)
At the start: 4 copper layers, 92.3 x 143 mm, 213 parts, among them J2 Value: DISP_3.5_WAVESHARE, P1 JST-2pin, P2 USB_C_Plug_USB2.0, Q1 MMBT2222A, Q2 FS8205A, SW1 boot, SW2 REST, SW3 BTN_POWER, SW4 BTN_OK, SW5 BTN_UP, SW6 BTN_DOWN, SW7 BTN_LEFT, SW8 BTN_RIGHT, U1 ESP32-S3, U10 BGA725L6, U11 TLV70018_SOT23-5, U12 TXB0102DCU, U13 MCP23017x-x-SS, U14 TSOP382xx, U15 TP4056, U16 PESD5V0L4UG,115, U17 AP2112K-3.3, U18 DW01A, U19 SX1262IMLTRT, U2 W25Q128JVS, U20 PE4259, U3 CC1101, U7 PN5321A3HN, U8 MAX-M8Q, U9 MASW-007221, Y1 40MHz SMD 3225, Y2 26 MHz SMD, Y4 27.120 MHz, Y5 32 MHz SMD

Commit message: yay
Parts:
- moved AE1 35.8 mm to (116.5, 98.8)
- moved R25 12.0 mm to (161.2, 104.8), turned to 0 degrees
- moved FL1 7.81 mm to (166.9, 104.0), turned to 180 degrees
- moved R24 6.56 mm to (170.2, 107.0)
- moved C91 6.25 mm to (164.0, 104.5), turned to 0 degrees
- moved C92 5.82 mm to (172.5, 104.0), turned to 180 degrees
- moved JP1 5.60 mm to (161.8, 101.3), turned to 0 degrees
- moved C100 5.11 mm to (159.0, 101.6)
- moved C89 5.11 mm to (168.5, 101.0)
- moved FB1 4.50 mm to (165.8, 101.1)
- moved U10 4.23 mm to (169.2, 104.0), turned to -90 degrees
- moved U9 4.22 mm to (171.8, 101.3)
- moved C94 3.74 mm to (177.1, 113.2), turned to 0 degrees
- moved C95 3.25 mm to (173.8, 130.2), turned to 0 degrees
- moved C98 2.83 mm to (159.0, 105.4)
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
Commit message: uug
Parts:
- moved AE1 11.1 mm to (127.5, 100.5)
Routing:
- removed copper zone on In1.Cu, net GND
- removed copper zone on In2.Cu, net VDD33
Other:
- board size 92.3 x 143 mm -> 142.1 x 143 mm
Changed lines of the file:
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@@
 	(footprint "KiCad_Package coil:NFC_45x45_N4_NXP_PN5180"
 		(layer "B.Cu")
-		(at 116.55 98.75)
+		(at 127.5 100.5)
 		(property "Reference" "AE1"
 			(at 0 0 0)
@@
 		)
 		(property "Value" "PN532 ANT"
-			(at 0 0 0)
+			(at 0 -4.75 0)
 			(layer "B.Fab")
 			(effects
@@
 	)
 	(gr_line
-		(start 152.358922 71.294591)
-		(end 152.358922 126.472536)
+		(start 102.549349 78.612115)
+		(end 102.549349 122.362115)
+		(stroke
+			(width 0.05)
+			(type default)
+		)
+		(layer "Edge.Cuts")
+	)
+	(gr_arc
+		(start 102.549349 78.612115)
+		(mid 103.486817 76.348947)
+		(end 105.75 75.411517)
+		(stroke
+			(width 0.05)
+			(type default)
+		)
+		(layer "Edge.Cuts")
+	)
+	(gr_arc
+		(start 105.661518 125.474271)
+		(mid 103.460887 124.562742)
+		(end 102.549349 122.362115)
+		(stroke
+			(width 0.05)
+			(type default)
+		)
+		(layer "Edge.Cuts")
+	)
+	(gr_line
+		(start 105.661518 125.474271)
+		(end 152.358922 125.474271)
+		(stroke
+			(width 0.05)
+			(type default)
+		)
+		(layer "Edge.Cuts")
+	)
+	(gr_line
+		(start 149.246766 75.411517)
+		(end 105.75 75.411517)
 		(stroke
 			(width 0.05)
@@
 		(layer "Edge.Cuts")
 	)
+	(gr_line
+		(start 152.358922 71.2946)
+		(end 152.358922 72.299401)
+		(stroke
+			(width 0.05)
+			(type default)
+		)
+		(layer "Edge.Cuts")
+	)
+	(gr_arc
+		(start 152.358922 72.299401)
+		(mid 151.447373 74.5)
+		(end 149.246766 75.411517)
+		(stroke
+			(width 0.05)
+			(type default)
+		)
+		(layer "Edge.Cuts")
+	)
+	(gr_line
+		(start 152.358922 126.472536)
+		(end 152.358922 125.48)
+		(stroke
+			(width 0.05)
+			(type solid)
+		)
+		(layer "Edge.Cuts")
+	)
 	(gr_arc
 		(start 155.471038 129.584692)
@@
 			(type default)
 		)
-		(locked yes)
 		(layer "Edge.Cuts")
 	)
@@
 			(type default)
 		)
-		(locked yes)
 		(layer "Edge.Cuts")
 	)
@@
 		(layer "Edge.Cuts")
 	)
-	(zone
-		(net "GND")
-		(layer "In1.Cu")
-		(hatch edge 0.5)
-		(connect_pads yes
-			(clearance 0.5)
-		)
-		(min_thickness 0.25)
-		(fill yes
-			(thermal_gap 0.4)
-			(thermal_bridge_width 0.5)
-			(island_removal_mode 0)
-		)
-		(polygon
-			(pts
-				(xy 239 68.25) (xy 241.75 68.25) (xy 243 68.5) (xy 244.25 69.75) (xy 244.5 70.5) (xy 244.5 127.75)
-				(xy 244.25 128.25) (xy 243.75 129) (xy 243.5 129.25) (xy 241.75 130) (xy 241 130) (xy 240.25 130.25)
-				(xy 239.75 130.5) (xy 239 131) (xy 238.25 132.25) (xy 238 134.5) (xy 238 185) (xy 241.5 185) (xy 241.5 195.75)
-				(xy 238 195.75) (xy 238 207.75) (xy 237.5 209.25) (xy 236.75 210.25) (xy 235.25 211) (xy 161.25 211)
-				(xy 160.089286 210.616071) (xy 158.910715 209.633929) (xy 158.5 209) (xy 158.5 208.75) (xy 158.5 133)
-				(xy 157.958333 130.958333) (xy 157.25 130.25) (xy 156.25 129.75) (xy 155.25 129.5) (xy 154.75 129.5)
-				(xy 153.75 129) (xy 152.75 128) (xy 152.5 127.25) (xy 152.5 70.5) (xy 152.75 69.75) (xy 154 68.5)
-				(xy 155.5 68)
-			)
-		)
-	)
-	(zone
-		(net "VDD33")
-		(layer "In2.Cu")
-		(hatch edge 0.5)
-		(priority 1)
-		(connect_pads yes
-			(clearance 0.5)
-		)
-		(min_thickness 0.25)
-		(fill yes
-			(thermal_gap 0.4)
-			(thermal_bridge_width 0.5)
-			(island_removal_mode 0)
-		)
-		(polygon
-			(pts
-				(xy 243 68.5) (xy 241.75 68.25) (xy 155.5 68) (xy 154 68.5) (xy 152.75 69.75) (xy 152.5 70.5) (xy 152.5 127.25)
-				(xy 152.75 128) (xy 153.75 129) (xy 154.75 129.5) (xy 155.25 129.5) (xy 156.25 129.75) (xy 157.25 130.25)
-				(xy 158 131) (xy 158.5 133) (xy 158.5 209) (xy 159 209.75) (xy 159.5 210.25) (xy 160.25 210.75)
-				(xy 161.25 211) (xy 235.25 211) (xy 236.75 210.25) (xy 237.5 209.25) (xy 238 207.75) (xy 238 195.75)
-				(xy 241.5 195.75) (xy 241.5 185) (xy 238 185) (xy 238 134.5) (xy 238.25 132.25) (xy 239 131) (xy 240.5 130)
-				(xy 241.75 130) (xy 243.5 129.25) (xy 243.75 129) (xy 244.25 128.25) (xy 244.5 127.5) (xy 244.5 70.5)
-				(xy 244.25 69.75)
-			)
-		)
-	)
 	(embedded_fonts no)
