File: PCB/Flipper black ki cad/Flipper black ki cad.kicad_pcb (KiCad board)
At the start: 4 copper layers, 142.1 x 143 mm, 217 parts, among them J2 Value: DISP_3.5_WAVESHARE, P1 JST-2pin, P2 USB_C_Plug_USB2.0, Q1 MMBT2222A, Q2 FS8205A, SW1 boot, SW2 REST, SW3 BTN_POWER, SW4 BTN_OK, SW5 BTN_UP, SW6 BTN_DOWN, SW7 BTN_LEFT, SW8 BTN_RIGHT, U1 ESP32-S3, U10 BGA725L6, U11 TLV70018_SOT23-5, U12 TXB0102DCU, U13 MCP23017x-x-SS, U14 TSOP382xx, U15 TP4056, U16 PESD5V0L4UG,115, U17 AP2112K-3.3, U18 DW01A, U19 SX1262IMLTRT, U2 W25Q128JVS, U20 PE4259, U3 CC1101, U7 PN5321A3HN, U8 MAX-M8Q, U9 MASW-007221, Y1 40MHz SMD 3225, Y2 26 MHz SMD, Y4 27.120 MHz, Y5 32 MHz SMD

Commit message: jjmario
Routing:
- net Net-(SX1262-A): track 89.5 -> 93.8 mm
Changed lines of the file:
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@@
 	)
 	(segment
-		(start 152.7675 111.238924)
-		(end 152.7675 111.2)
+		(start 139.4 106.4)
+		(end 139.4 82.2)
 		(width 0.2)
 		(layer "F.Cu")
@@
 	)
 	(segment
-		(start 152.7675 111.2)
-		(end 138.6 97.0325)
+		(start 170.525 113.175)
+		(end 146.175 113.175)
+		(width 0.2)
+		(layer "F.Cu")
+		(net "Net-(SX1262-A)")
+	)
+	(segment
+		(start 141.6 80)
+		(end 154.540256 80)
 		(width 0.2)
 		(layer "F.Cu")
@@
 	)
 	(segment
-		(start 138.6 97.0325)
-		(end 138.6 83)
+		(start 146.175 113.175)
+		(end 139.4 106.4)
 		(width 0.2)
 		(layer "F.Cu")
@@
 	)
 	(segment
-		(start 154.703576 113.175)
-		(end 152.7675 111.238924)
-		(width 0.2)
-		(layer "F.Cu")
-		(net "Net-(SX1262-A)")
-	)
-	(segment
-		(start 138.6 83)
+		(start 139.4 82.2)
 		(end 141.6 80)
-		(width 0.2)
-		(layer "F.Cu")
-		(net "Net-(SX1262-A)")
-	)
-	(segment
-		(start 162.465256 72.075)
-		(end 164.325 72.075)
-		(width 0.2)
-		(layer "F.Cu")
-		(net "Net-(SX1262-A)")
-	)
-	(segment
-		(start 141.6 80)
-		(end 154.540256 80)
 		(width 0.2)
 		(layer "F.Cu")
@@
 	)
 	(segment
-		(start 170.525 113.175)
-		(end 154.703576 113.175)
+		(start 162.465256 72.075)
+		(end 164.325 72.075)
 		(width 0.2)
 		(layer "F.Cu")
