File: PCB/Flipper black ki cad/Flipper black ki cad.kicad_sch (KiCad schematic)
At the start: 213 parts, among them J2 Value: DISP_3.5_WAVESHARE, P1 JST-2pin, P2 USB_C_Plug_USB2.0, Q1 MMBT2222A, Q2 FS8205A, SW1 boot, SW2 REST, SW3 BTN_POWER, SW4 BTN_OK, SW5 BTN_UP, SW6 BTN_DOWN, SW7 BTN_LEFT, SW8 BTN_RIGHT, U1 ESP32-S3, U10 BGA725L6, U11 TLV70018_SOT23-5, U12 TXB0102DCU, U13 MCP23017x-x-SS, U14 TSOP382xx, U15 TP4056, U16 PESD5V0L4UG,115, U17 AP2112K-3.3, U18 DW01A, U19 SX1262IMLTRT, U2 W25Q128JVS, U20 PE4259, U3 CC1101, U7 PN5321A3HN, U8 MAX-M8Q, U9 MASW-007221, Y1 40MHz SMD 3225, Y2 26 MHz SMD, Y4 27.120 MHz, Y5 32 MHz SMD

Commit message: jjmario
Parts:
- added J1: Micro_SD_Card_Det2, symbol Connector:Micro_SD_Card_Det2
Other:
- note added: "Micro SD Card"
Changed lines of the file:
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@@
 		)
 	)
+	(text "Micro SD Card"
+		(exclude_from_sim no)
+		(at 76.2 443.484 0)
+		(effects
+			(font
+				(size 2.54 2.54)
+				(thickness 0.508)
+				(bold yes)
+			)
+		)
+	)
 	(text "CC1101 - Sub-GHz Transceiver"
 		(exclude_from_sim no)
@@
 		)
 	)
+	(polyline
+		(pts
+			(xy 60.96 447.04) (xy 91.44 447.04)
+		)
+		(stroke
+			(width 1)
+			(type solid)
+		)
+	)
 	(wire
 		(pts
@@
 		)
 	)
+	(polyline
+		(pts
+			(xy 91.44 447.04) (xy 91.44 439.928)
+		)
+		(stroke
+			(width 1)
+			(type solid)
+		)
+	)
 	(wire
 		(pts
@@
 	(polyline
 		(pts
+			(xy 15.24 439.42) (xy 15.24 508)
+		)
+		(stroke
+			(width 1)
+			(type solid)
+		)
+	)
+	(polyline
+		(pts
 			(xy 695.96 68.58) (xy 695.96 15.24)
 		)
@@
 		)
 	)
+	(polyline
+		(pts
+			(xy 142.24 439.42) (xy 142.24 508)
+		)
+		(stroke
+			(width 1)
+			(type solid)
+		)
+	)
 	(wire
 		(pts
@@
 	(polyline
 		(pts
+			(xy 142.24 508) (xy 15.24 508)
+		)
+		(stroke
+			(width 1)
+			(type solid)
+		)
+	)
+	(polyline
+		(pts
 			(xy 695.96 205.74) (xy 746.76 205.74)
 		)
@@
 		)
 	)
+	(polyline
+		(pts
+			(xy 60.96 439.928) (xy 60.96 447.04)
+		)
+		(stroke
+			(width 1)
+			(type solid)
+		)
+	)
 	(wire
 		(pts
@@
 	(polyline
 		(pts
+			(xy 15.24 439.42) (xy 142.24 439.42)
+		)
+		(stroke
+			(width 1)
+			(type solid)
+		)
+	)
+	(polyline
+		(pts
 			(xy 439.42 345.44) (xy 439.42 353.06)
 		)
@@
 					(unit 1)
 				)
+			)
+		)
+	)
+	(symbol
+		(lib_id "Connector:Micro_SD_Card_Det2")
+		(at 76.2 477.52 0)
+		(unit 1)
+		(body_style 1)
+		(exclude_from_sim no)
+		(in_bom yes)
+		(on_board yes)
+		(in_pos_files yes)
+		(dnp no)
+		(fields_autoplaced yes)
+		(property "Reference" "J1"
+			(at 76.835 455.93 0)
+			(show_name no)
+			(do_not_autoplace no)
+			(effects
+				(font
+					(size 1.27 1.27)
+				)
+			)
+		)
+		(property "Value" "Micro_SD_Card_Det2"
+			(at 76.835 458.47 0)
+			(show_name no)
+			(do_not_autoplace no)
+			(effects
+				(font
+					(size 1.27 1.27)
+				)
+			)
+		)
+		(property "Footprint" ""
+			(at 128.27 459.74 0)
+			(hide yes)
+			(show_name no)
+			(do_not_autoplace no)
+			(effects
+				(font
+					(size 1.27 1.27)
+				)
+			)
+		)
+		(property "Datasheet" "https://www.hirose.com/en/product/document?clcode=&productname=&series=DM3&documenttype=Catalog&lang=en&documentid=D49662_en"
+			(at 78.74 474.98 0)
+			(hide yes)
+			(show_name no)
+			(do_not_autoplace no)
+			(effects
+				(font
+					(size 1.27 1.27)
+				)
+			)
+		)
+		(property "Description" "Micro SD Card Socket with two card detection pins"
+			(at 76.2 477.52 0)
+			(hide yes)
+			(show_name no)
+			(do_not_autoplace no)
+			(effects
+				(font
+					(size 1.27 1.27)
+				)
+			)
+		)
+		(pin "5"
+		)
+		(pin "8"
+		)
+		(pin "2"
+		)
+		(pin "7"
+		)
+		(pin "1"
+		)
+		(pin "3"
+		)
+		(pin "6"
+		)
+		(pin "4"
+		)
+		(pin "SH"
+		)
+		(pin "10"
+		)
+		(pin "9"
+		)
+		(instances
+			(project "Flipper black ki cad"
+				(path "/aadf5baa-c41c-48f9-af5f-e274c89cf282"
+					(reference "J1")
+					(unit 1)
+				)

Commit message: yayay
Parts:
- added C29: 100nf, Capacitor_SMD:C_0603_1608Metric_Pad1.08x0.95mm_HandSolder, symbol Device:C
- added R8: 10K, Resistor_SMD:R_0402_1005Metric, symbol Device:R
- J1: footprint (none) -> MEM2067-02-180-00-A_REVB:GCT_MEM2067-02-180-00-A_REVB
Connections:
- net GND: now also J1.6 (VSS), J1.9 (DET_B), J1.SH (SHIELD), C29.2
- net SPI_MISO: now also J1.7 (DAT0)
- net SPI_MOSI: now also J1.3 (CMD)
- net SPI_SCK: now also J1.5 (CLK)
- net VDD33: now also J1.4 (VDD), C29.1, R8.2
- net SD_CS: now reaches U13.1 (GPB0)
- net SD_CS: now also J1.2 (DAT3/CD)
- net SD_CD: now reaches U13.2 (GPB1)
- net SD_CD: now also J1.10 (DET_A), R8.1
- no-connect marks 21 -> 22
Other:
- moved on the sheet: J1
